File: tac5212_audio_board_single_ended.kicad_pcb (KiCad board)
At the start: 4 copper layers, 42 x 26.5 mm, 99 parts, among them J10 Conn_02x08_Odd_Even, J1002 TAC5212, J2 Conn_02x08_Odd_Even, J3 Conn_02x08_Odd_Even, J4 HEADPHONE, J5 HEADPHONE, J6 Conn_02x08_Odd_Even, J7 Conn_02x08_Odd_Even, J8 Conn_02x08_Odd_Even, J9 Conn_02x08_Odd_Even, U1 Single Buffer - 74LVC1G125GV,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, U2 3.3v LDO - TLV74133PDQNR

Commit message: update
Parts:
- removed BAL_IN1: NCJ6FA, project_fp:Jack_XLR-6.35mm_Neutrik_NCJ6FA-H-0_Horizontal
- removed BYPASS1, BYPASS2, BYPASS3, BYPASS4: jumper, project_fp:SolderJumper-2_P1.3mm_Bridged2Bar_RoundedPad1.0x1.5mm_OPEN
- removed GPIO1001: Conn_01x05_Pin, Connector_PinHeader_2.54mm:PinHeader_1x05_P2.54mm_Vertical
- removed HPTRS1, HPTRS2: 3.5MM JACK, project_fp:35RAPC3BH3
- removed J10, J9: Conn_02x08_Odd_Even, Connector_PinHeader_2.54mm:PinHeader_2x04_P2.54mm_Vertical
- removed J2, J3: Conn_02x08_Odd_Even, Connector_IDC:IDC-Header_2x04_P2.54mm_Vertical
- removed J4, J5: HEADPHONE, project_fp:PinHeader_2x02_P2.54mm_Vertical
- removed J6: Conn_02x08_Odd_Even, Connector_IDC:IDC-Header_2x08_P2.54mm_Vertical
- removed J7, J8: Conn_02x08_Odd_Even, Connector_PinHeader_2.54mm:PinHeader_1x04_P2.54mm_Vertical
- removed JHP1, JHP3: JHP1, project_fp:SolderJumper-3_P1.3mm_Bridged12_Pad1.0x1.5mm_NO_REF
- removed JHP2, JHP4: JHP2, project_fp:SolderJumper-3_P1.3mm_Bridged12_Pad1.0x1.5mm_NO_REF
- removed LINE_IO1: 3.5mm Dual - 35RAPC7JS, project_fp:35RAPC7JS
- removed OUTL1, OUTR1: jumper, project_fp:SolderJumper-3_P_12_BRIDGED
- removed PD3.1: header, project_fp:PinHeader_1x01_P2.54mm_Vertical
- removed R6: 0 Ohm, Resistor_SMD:R_0402_1005Metric_Pad0.72x0.64mm_HandSolder
- removed RCA_IN1: RCA 2X2 - PJRAS2X2S01AUX, project_fp:PJRAS2X2S01AUX
- removed TRS1, TRS2: 35RAPC3BH3, project_fp:Jack_6.35mm_Neutrik_NMJ6HCD3_Horizontal
- removed XIA1: header, project_fp:T-DSP_Expansion_Header_2x10_ALT_GND
- removed XIA2: header, Connector_PinHeader_2.54mm:PinHeader_1x12_P2.54mm_Vertical
- added IN1: Jump Filter, project_fp:jumper_slice_via, B.Cu at (124.8, 107.2)
- added IN2: Jump Filter, project_fp:jumper_slice_via, B.Cu at (121.5, 107.2)
- added IN3: Jump Filter, project_fp:jumper_slice_via, B.Cu at (118.2, 107.1)
- added IN4: Jump Filter, project_fp:jumper_slice_via, B.Cu at (114.9, 107.1)
- added OUT1: Jump Filter, project_fp:jumper_slice_via, B.Cu at (95.8, 107.0)
- added OUT2: Jump Filter, project_fp:jumper_slice_via, B.Cu at (92.0, 107.0)
- added OUT3: Jump Filter, project_fp:jumper_slice_via, B.Cu at (99.6, 107.0)
- added OUT4: Jump Filter, project_fp:jumper_slice_via, B.Cu at (103.3, 107.0)
- MCLK1: footprint project_fp:jumper_slice -> project_fp:jumper_slice_disconnected; moved to B.Cu
- moved ADD1001 6.69 mm to (118.2, 111.0), turned to -90 degrees
- moved ADD1002 4.96 mm to (119.6, 111.0), turned to 90 degrees
- moved PU_EN1001 3.77 mm to (124.1, 111.0), turned to -90 degrees
- moved ADD1003 3.48 mm to (121.1, 111.0), turned to 90 degrees
- moved R1001 3.18 mm to (120.4, 114.0), turned to -90 degrees
- moved ADD1004 2.94 mm to (122.6, 110.9), turned to 90 degrees
- moved R1003 2.93 mm to (124.3, 114.0), turned to -90 degrees
- moved C1011 1.47 mm to (113.7, 111.8)
- moved FB1004 1.34 mm to (113.4, 107.9)
- moved R1002 1.32 mm to (122.3, 114.0), turned to -90 degrees
- moved SCL1001 1.20 mm to (92.8, 101.4)
- moved C1015 1.18 mm to (100.7, 116.7)
- moved C1001 1.12 mm to (102.1, 110.2)
- moved C1002 1.12 mm to (107.8, 118.4)
- moved C1005 1.12 mm to (104.6, 112.2)
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Connections:
- net 5212_SCL_A renamed DSP_SCL
- net 5212_SDA_A renamed DSP_SDA
- SCL1001 pad 2: unconnected-(SCL1001-B-Pad2) -> 5212_SCL
- SDA1001 pad 2: unconnected-(SDA1001-B-Pad2) -> 5212_SDA
- board_outline1 pad 22: AUX2L -> PHONE1L
- board_outline1 pad 24: AUX2R -> PHONE1R
- board_outline1 pad 26: AUX1L -> RCAL
- board_outline1 pad 28: AUX1R -> RCAR
- board_outline1 pad 30: PHONE1L -> AUX1L
- board_outline1 pad 32: PHONE1R -> AUX1R
- board_outline1 pad 34: RCAL -> AUX2L
- board_outline1 pad 36: RCAR -> AUX2R
Routing:
- net 5V: track 0.00 -> 41.0 mm, vias 0 -> 1
- net 5212_SCL: track 16.0 -> 56.0 mm, vias 0 -> 1
- net 5212_SDA: track 15.4 -> 47.4 mm, vias 0 -> 2
- net Net-(J1002-ADDR): track 0.00 -> 21.9 mm, vias 0 -> 2
- net PHONE1R: track 0.00 -> 21.2 mm
- net OUT1M: track 16.2 -> 31.1 mm, vias 1 -> 0
- net OUT1P: track 11.8 -> 26.3 mm, vias 1 -> 0
- net RCAR: track 0.00 -> 14.1 mm
- net PHONE1L: track 0.00 -> 13.9 mm
- net OUT2P: track 7.67 -> 21.4 mm, vias 1 -> 0
- net OUT2M: track 3.11 -> 16.6 mm, vias 1 -> 0
- net RCAL: track 0.00 -> 13.4 mm
- net AUX2R: track 0.00 -> 9.31 mm
- net AUX2L: track 0.00 -> 8.56 mm
- net AUX1R: track 0.00 -> 7.71 mm
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
Commit message: update
Parts:
- added SCL1: jumper, project_fp:jumper_slice, B.Cu at (109.2, 107.3)
Connections:
- D1002 pad 2: unconnected-(D1002-K-Pad2) -> Earth
- D1003 pad 2: unconnected-(D1003-K-Pad2) -> Earth
- D1004 pad 2: unconnected-(D1004-K-Pad2) -> Earth
- D1005 pad 2: unconnected-(D1005-K-Pad2) -> Earth
- D1006 pad 2: unconnected-(D1006-K-Pad2) -> Earth
- J1002 pad 25: Earth -> GNDD
- board_outline1 pad 21: unconnected-(board_outline1-Pin_21-Pad21) -> Earth
- board_outline1 pad 23: unconnected-(board_outline1-Pin_23-Pad23) -> Earth
- board_outline1 pad 25: unconnected-(board_outline1-Pin_25-Pad25) -> Earth
- board_outline1 pad 27: unconnected-(board_outline1-Pin_27-Pad27) -> Earth
- board_outline1 pad 29: unconnected-(board_outline1-Pin_29-Pad29) -> Earth
- board_outline1 pad 31: unconnected-(board_outline1-Pin_31-Pad31) -> Earth
- board_outline1 pad 33: unconnected-(board_outline1-Pin_33-Pad33) -> Earth
- board_outline1 pad 35: unconnected-(board_outline1-Pin_35-Pad35) -> Earth
Routing:
- net Net-(PU_EN1001-Pad2): track 2.48 -> 29.0 mm, vias 1 -> 2
- net GNDD: track 0.00 -> 1.71 mm
- net Earth: vias 0 -> 13
- added copper zone on B.Cu, net Earth
- added copper zone on In2.Cu, net Earth
- added copper zone on F.Cu, net GNDD
- added copper zone on In1.Cu, net GNDD
Other:
- outline, holes or cut-outs redrawn
