File: tac5212_audio_board_single_ended.kicad_pcb (KiCad board)
At the start: 4 copper layers, 42 x 26.5 mm, 93 parts, among them J1002 TAC5212, U1 Single Buffer - 74LVC1G125GV,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, U2 3.3v LDO - TLV74133PDQNR

Commit message: update
Parts:
- OM1: footprint project_fp:jumper_slice_via -> project_fp:jumper_slice_via_alt_text
- moved G10 7.81 mm to (125.9, 110.2)
- moved G9 4.00 mm to (103.2, 119.3)
- moved R1001 1.50 mm to (116.7, 112.2)
- moved R1002 1.50 mm to (119.1, 112.2)
- moved ADD1004 1.50 mm to (121.6, 110.2)
- moved R1003 1.40 mm to (121.4, 112.2)
- moved ADD1003 1.20 mm to (120.2, 110.2)
- moved R5 1.14 mm to (120.3, 115.1)
- moved D7 1.14 mm to (119.7, 117.3)
- moved C1 1.00 mm to (96.8, 118.0)
- moved ADD1002 0.90 mm to (118.8, 110.2)
- moved R1 0.76 mm to (96.5, 111.8)
- moved G7 0.51 mm to (102.6, 118.4)
- moved ADD1001 0.50 mm to (117.4, 110.2)
- moved C1006 0.35 mm to (105.1, 109.2)
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Connections:
- C1001 pad 1: AVDD -> 3.3V_LDO
Routing:
- net GNDD: track 3.87 -> 47.1 mm, vias 0 -> 4
- net Net-(E1-A): track 5.99 -> 28.9 mm
- net Earth: track 148.1 -> 157.4 mm
- net /GPI1: track 77.7 -> 70.3 mm
- net AVDD: track 5.14 -> 0.00 mm
- net 3.3V_LDO: track 83.2 -> 87.9 mm, vias 2 -> 3
- net DSP_SDA: track 0.00 -> 3.15 mm
- net Net-(J1002-ADDR): track 12.0 -> 10.5 mm
- net OUT1M: track 30.0 -> 31.0 mm
- net 5212_DOUT1+: track 14.3 -> 15.3 mm
- net Net-(U1-Y): track 2.80 -> 3.61 mm

Commit message: update
Connections:
- E1 pad 1: Net-(E1-A) -> unconnected-(E1-A-Pad1)
- E2 pad 1: Net-(E1-A) -> unconnected-(E2-A-Pad1)
- G1 pad 1: Net-(G1-A) -> unconnected-(G1-A-Pad1)
- G2 pad 1: Net-(G1-A) -> unconnected-(G2-A-Pad1)
- board_outline1 pad 49: Net-(E1-A) -> unconnected-(board_outline1-AGND-Pad49)
- board_outline1 pad 50: Net-(G1-A) -> unconnected-(board_outline1-AGND-Pad50)
- board_outline1 pad 51: (no net) -> unconnected-(board_outline1-DGND-Pad51)
- board_outline1 pad 52: (no net) -> unconnected-(board_outline1-DGND-Pad52)
Routing:
- net (no net): track 0.00 -> 34.4 mm
- net Net-(E1-A): track 28.9 -> 0.00 mm
- net Net-(G1-A): track 5.53 -> 0.00 mm

Commit message: update
Parts:
- added ADD1: jumper, project_fp:SolderJumper-2_Open_Pad0.5x1.0mm_ADDR, F.Cu at (122.2, 111.0)
- C1, T*C2: footprint project_fp:C_0805_2012Metric_Pad1.18x1.45mm_HandSolder -> Capacitor_SMD:C_0603_1608Metric_Pad1.08x0.95mm_HandSolder
- C10: renamed from C1003; footprint Capacitor_SMD:C_0805_2012Metric -> project_fp:C_0805_2012Metric_Pad1.18x1.45mm_HandSolder
- C1009, C1010, C1011: value 0.1UF - 100V Ceramic Chip Capacitor, ±10%, X7R -> 10UF
- C1012: value CAP CER 4.7UF 50V X7R 1206 - CAP ALUM 4.7UF 20% 50V RADIAL -> 10UF
- C12: renamed from C1002; footprint Capacitor_SMD:C_0805_2012Metric -> project_fp:C_0805_2012Metric_Pad1.18x1.45mm_HandSolder
- C13: renamed from C1001; footprint project_fp:C_0805_2012Metric -> project_fp:C_0805_2012Metric_Pad1.18x1.45mm_HandSolder
- C17: renamed from C1004; footprint Capacitor_SMD:C_0603_1608Metric -> Capacitor_SMD:C_0603_1608Metric_Pad1.08x0.95mm_HandSolder
- C18: renamed from C1013; value 47UF CAP CER 6.3V X5R 1210 - 47uF Radial -> 47uF
- C19: renamed from C1014; value 47UF CAP CER 6.3V X5R 1210 - 47uF Radial -> 47uF
- C20: renamed from C1015; value 47UF CAP CER 6.3V X5R 1210 - 47uF Radial -> 47uF
- C21: renamed from C1016; value 47UF CAP CER 6.3V X5R 1210 - 47uF Radial -> 47uF
- C22: renamed from C1019; value 47NF CAP CER 100V X7R 0805 -> 0.047uF; footprint project_fp:C_0805_2012Metric_Pad1.18x1.45mm_HandSolder -> Capacitor_SMD:C_0603_1608Metric_Pad1.08x0.95mm_HandSolder
- C23: renamed from C1017; value 47NF CAP CER 100V X7R 0805 -> 0.047uF; footprint project_fp:C_0805_2012Metric_Pad1.18x1.45mm_HandSolder -> Capacitor_SMD:C_0603_1608Metric_Pad1.08x0.95mm_HandSolder
- C24: renamed from C1018; value 47NF CAP CER 100V X7R 0805 -> 0.047uF; footprint project_fp:C_0805_2012Metric_Pad1.18x1.45mm_HandSolder -> Capacitor_SMD:C_0603_1608Metric_Pad1.08x0.95mm_HandSolder
- C25: renamed from C1020; value 47NF CAP CER 100V X7R 0805 -> 0.047uF; footprint project_fp:C_0805_2012Metric_Pad1.18x1.45mm_HandSolder -> Capacitor_SMD:C_0603_1608Metric_Pad1.08x0.95mm_HandSolder
- D7: value LED - B2601USD-20D000423U1930 -> RED LED; footprint project_fp:LED_1206_3216Metric_Pad1.42x1.75mm_HandSolder -> project_fp:R_0805_2012Metric_Pad1.20x1.40mm_HandSolder
- R1: footprint project_fp:R_0805_2012Metric_Pad1.20x1.40mm_HandSolder -> Resistor_SMD:R_0402_1005Metric_Pad0.72x0.64mm_HandSolder
- R17: renamed from R1015; value 100ohm -> 100; footprint project_fp:R_0805_2012Metric_Pad1.20x1.40mm_HandSolder -> project_fp:R_0603_1608Metric_Pad1.05x0.95mm_HandSolder
- R18: renamed from R1018; value 100ohm -> 100; footprint project_fp:R_0805_2012Metric_Pad1.20x1.40mm_HandSolder -> project_fp:R_0603_1608Metric_Pad1.05x0.95mm_HandSolder
- R19: renamed from R1016; value 1K RES SMD OHM 1% 1/2W 0805 -> 100; footprint project_fp:R_0805_2012Metric_Pad1.20x1.40mm_HandSolder -> project_fp:R_0603_1608Metric_Pad1.05x0.95mm_HandSolder
- R20: renamed from R1017; value 1K RES SMD OHM 1% 1/2W 0805 -> 100; footprint project_fp:R_0805_2012Metric_Pad1.20x1.40mm_HandSolder -> project_fp:R_0603_1608Metric_Pad1.05x0.95mm_HandSolder
- R40: renamed from R1001; value 4.7KOhm -> 4.7k
- R41: renamed from R1003; value 4.7KOhm -> 4.7k
- R42: renamed from R1002; value 22KOhm -> 22.0k
- R5: footprint project_fp:R_0805_2012Metric_Pad1.20x1.40mm_HandSolder -> Resistor_SMD:R_0402_1005Metric
- T*C1, T*C3: value DNP (10uF) -> 10uF
- U2: value 3.3v LDO - TLV74133PDQNR -> 3.3v LDO - TLV74133PDBVR
- moved R5 2.62 mm to (122.2, 116.9), turned to -90 degrees
- moved R1 1.61 mm to (95.1, 112.6)
- moved ADD1001 1.06 mm to (116.6, 111.0)
- moved ADD1002 1.06 mm to (118.0, 111.0)
- moved ADD1003 1.06 mm to (119.4, 111.0)
- moved ADD1004 1.06 mm to (120.8, 111.0)
- moved R42 0.76 mm to (119.4, 112.9)
- moved R40 0.73 mm to (116.9, 112.9)
- moved R41 0.73 mm to (121.6, 112.9), turned to 0 degrees
- moved D7 0.54 mm to (120.2, 117.1), turned to -90 degrees
- moved C2 0.32 mm to (114.3, 108.8)
- moved G4 0.20 mm to (117.1, 114.0)
- moved G6 0.20 mm to (118.4, 114.0)
- renumbered C1005 to C11, C1007 to C14, C1006 to C15, C1008 to C2, D1006 to D17, D1008 to D18, D1009 to D19, D1007 to D20, R1005 to R100, R1006 to R101, R1007 to R102, R1008 to R103, R1010 to R104, R1011 to R105, R1012 to R106, R1013 to R107, R1004 to R108, R1009 to R109
Connections:
- net /DSP_5V renamed Net-(5V1-B)
- net /GPI1 renamed GPI1
- net /GPIO1 renamed GPIO1
- net /GPIO2 renamed GPIO2
- net /GPO1 renamed GPO1
- net DREG renamed Net-(J1002-DREG)
- E1 pad 1: unconnected-(E1-A-Pad1) -> Net-(E1-A)
- E2 pad 1: unconnected-(E2-A-Pad1) -> Net-(E2-A)
- G1 pad 1: unconnected-(G1-A-Pad1) -> Net-(G1-A)
- G2 pad 1: unconnected-(G2-A-Pad1) -> Net-(G2-A)
- board_outline1 pad 1: /DSP_HELD_HIGH -> unconnected-(board_outline1-HELD_HIGH-Pad1)
- board_outline1 pad 2: GNDD -> unconnected-(board_outline1-HELD_LOW-Pad2)
- board_outline1 pad 49: unconnected-(board_outline1-AGND-Pad49) -> Net-(E1-A)
- board_outline1 pad 5: /DSP_12V -> unconnected-(board_outline1-12V-Pad5)
- board_outline1 pad 50: unconnected-(board_outline1-AGND-Pad50) -> Net-(E2-A)
- board_outline1 pad 51: unconnected-(board_outline1-DGND-Pad51) -> Net-(G1-A)
- board_outline1 pad 52: unconnected-(board_outline1-DGND-Pad52) -> Net-(G2-A)
Routing:
- net (no net): track 34.4 -> 28.9 mm
- net GNDD: track 47.1 -> 42.7 mm, vias 4 -> 3
- net Net-(U1-Y): track 3.61 -> 0.00 mm
- net Net-(G2-A): track 0.00 -> 2.94 mm
- net Net-(G1-A): track 0.00 -> 2.59 mm
- net MICBIAS: track 26.5 -> 24.0 mm
- net 5212_DOUT1+: track 15.3 -> 12.9 mm
- net 3.3V_LDO: track 87.9 -> 90.1 mm
- net 5212_LRCK1: track 22.3 -> 20.9 mm
- net 5212_BCLK1: track 27.6 -> 26.5 mm
- net Net-(J1002-ADDR): track 10.5 -> 11.5 mm
- net Net-(ADD1002-Pad1): track 2.20 -> 1.54 mm
- net Net-(PU_EN1001-Pad1): track 11.6 -> 12.3 mm
- net Earth: track 157.4 -> 157.7 mm, vias 0 -> 1
