File: tac5212_audio_board_single_ended.kicad_pcb (KiCad board)
At the start: 4 copper layers, 42 x 26.5 mm, 105 parts, among them T108 Tab, T109 Tab, T110 Tab, T111 Tab, U108 Single Buffer with Tri-state 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, U109 3.3v LDO - TLV74133PDBVR

Commit message: update
Parts:
- added G120: VIA, project_fp:via, B.Cu at (101.0, 128.5)
- added G121: VIA, project_fp:via, B.Cu at (110.0, 131.5)
- added G122: VIA, project_fp:via, B.Cu at (103.0, 131.5)
- added G123: SMD ROUTING PAD, project_fp:SMD_ROUTING_PAD, B.Cu at (106.5, 105.5)
- added G124: VIA, project_fp:via, B.Cu at (106.0, 128.5)
- added INM1: VIA, project_fp:via, B.Cu at (118.9, 107.5)
- added INM2: VIA, project_fp:via, B.Cu at (124.9, 107.5)
- added INP1: VIA, project_fp:via, B.Cu at (115.8, 107.5)
- added INP2: VIA, project_fp:via, B.Cu at (121.4, 105.0)
- added OUTM1: VIA, project_fp:via, B.Cu at (94.2, 104.2)
- added OUTM2: VIA, project_fp:via, B.Cu at (107.0, 109.0)
- added OUTP1: VIA, project_fp:via, B.Cu at (98.8, 105.0)
- added OUTP2: VIA, project_fp:via, B.Cu at (103.2, 106.5)
- C129: value 1uF -> 1uF is this the right value?
- G108, G109, G110, G111, G112, G113, G114, G115, G116: moved to B.Cu
- moved G115 88.9 mm to (120.9, 118.5), turned to 180 degrees
- moved G113 74.4 mm to (114.9, 118.5), turned to 180 degrees
- moved G110 62.5 mm to (101.5, 118.0), turned to 180 degrees
- moved G112 59.0 mm to (105.2, 118.0), turned to 180 degrees
- moved G109 57.3 mm to (93.2, 118.0), turned to 180 degrees
- moved G111 53.3 mm to (97.5, 118.0), turned to 180 degrees
- moved G114 46.8 mm to (117.9, 118.5), turned to 180 degrees
- moved G108 42.7 mm to (125.0, 106.0), turned to 180 degrees
- moved C130 10.5 mm to (93.0, 127.5)
- moved G116 8.54 mm to (123.9, 118.5), turned to 180 degrees
- moved C124 0.90 mm to (123.7, 116.5)
- moved C125 0.90 mm to (120.7, 116.5)
- moved C126 0.90 mm to (117.7, 116.5)
- moved C127 0.90 mm to (114.7, 116.5)
- moved D112 0.90 mm to (123.5, 106.5)
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Connections:
- C110 pad 2: OUT1M+ -> OUT1P+
- C117 pad 2: OUT1P+ -> OUT1M+
- D108 pad 1: OUT1M+ -> OUT1P+
- D109 pad 1: OUT1P+ -> OUT1M+
- R109 pad 2: OUT1P -> OUT1M
- R111 pad 2: OUT1P -> OUT1M
- R116 pad 1: OUT1P+ -> OUT1M+
- R129 pad 1: OUT1M+ -> OUT1P+
- R131 pad 2: OUT1P -> OUT2P
- R132 pad 2: OUT1P -> OUT2P
- R134 pad 2: OUT1P -> OUT2M
- R135 pad 2: OUT1P -> OUT2M
Routing:
- net Earth: track 140.0 -> 238.9 mm, vias 8 -> 7
- net 5V: track 65.7 -> 16.8 mm
- net OUT1P: track 66.4 -> 25.8 mm
- net OUT1M: track 20.6 -> 32.5 mm
- net OUT2P: track 10.00 -> 17.8 mm
- net OUT1P+: track 12.6 -> 6.01 mm
- net OUT2M+: track 13.5 -> 7.92 mm
- net OUT2P+: track 13.3 -> 7.92 mm
- net OUT2M: track 5.21 -> 9.50 mm
- net IN2M: track 32.8 -> 28.6 mm, vias 1 -> 0
- net IN1P: track 17.6 -> 14.5 mm, vias 1 -> 0
- net IN1M: track 21.7 -> 19.3 mm, vias 1 -> 0
- net IN2P: track 27.8 -> 25.5 mm, vias 1 -> 0
- net IN2P+: track 3.80 -> 1.74 mm
- net OUT1M+: track 6.01 -> 7.92 mm
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
Commit message: update
Parts:
- removed G115, G120, G121, G122, G124, OUTM2: VIA, project_fp:via
- removed R128: 2.21k ohm, project_fp:R_0402_1005Metric
- removed SCL109: jumper, Resistor_SMD:R_0402_1005Metric_Pad0.72x0.64mm_HandSolder
- C129: value 1uF is this the right value? -> 0.1uF; footprint project_fp:C_0603_1608Metric_Pad1.08x0.95mm_HandSolder -> project_fp:C_0402_1005Metric
- C130: moved to F.Cu
- FB108, FB109, FB110, FB111: footprint project_fp:C_0805_2012Metric_Pad1.18x1.45mm_HandSolder_alt_location -> project_fp:C_0805_2012Metric_Pad1.18x1.45mm_HandSolder
- G108, G109, G110, G111, G112: footprint project_fp:via -> project_fp:SMD_ROUTING_PAD
- moved C129 33.9 mm to (123.0, 120.0), turned to 0 degrees
- moved C130 7.50 mm to (93.2, 120.0)
- moved NT108 7.43 mm to (118.0, 120.0), turned to 180 degrees
- moved NT109 3.49 mm to (101.5, 108.0)
- moved G114 3.00 mm to (120.5, 120.0)
- moved G112 2.93 mm to (102.5, 119.0)
- moved G113 2.28 mm to (116.0, 120.5)
- moved INM1 1.50 mm to (119.0, 106.0)
- moved G111 1.22 mm to (98.7, 118.0)
- moved G116 1.21 mm to (125.0, 119.0)
- moved 5V108 1.20 mm to (92.9, 122.5)
- moved OUTP2 0.70 mm to (102.9, 105.9)
- moved INP1 0.58 mm to (115.5, 108.0)
- moved OUTM1 0.46 mm to (94.5, 104.5)
- moved C127 0.40 mm to (114.3, 116.5)
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Routing:
- net Earth: track 238.9 -> 309.2 mm, vias 7 -> 10
- net GNDD: track 83.6 -> 122.0 mm, vias 6 -> 7
- net GPI1: track 74.6 -> 43.5 mm, vias 1 -> 2
- net OUT1M+: track 7.92 -> 22.2 mm
- net 5V: track 16.8 -> 30.0 mm, vias 0 -> 2
- net 3.3V_LDO: track 28.4 -> 38.5 mm, vias 0 -> 2
- net EN_HELD_HIGH: track 27.6 -> 37.0 mm, vias 0 -> 1
- net OUT1P+: track 6.01 -> 14.2 mm
- net OUT2P+: track 7.92 -> 15.0 mm
- net IN2M+: track 1.74 -> 7.95 mm
- net IN2P+: track 1.74 -> 7.57 mm
- net OUT2M+: track 7.92 -> 13.6 mm
- net IN1M+: track 1.74 -> 7.30 mm
- net IN1P+: track 1.74 -> 7.11 mm
- net Net-(PU_EN108-Pad1): track 2.65 -> 6.18 mm, vias 0 -> 2
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Other:
- board text removed: "${Label}"
