File: tac5212_audio_board_single_ended.kicad_sch (KiCad schematic)
At the start: 78 parts, among them J1002 TAC5212, U1 Single Buffer - 74LVC1G125GV,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, U2 3.3v LDO - TLV74133PDQNR

Commit message: update
Parts:
- added 3V3, 5V1: jumper, project_fp:jumper_slice_1mm, symbol proejct_lib:Jumper_2_Bridged
- ADD1001: Label A1 -> 50
- ADD1002: Label A2 -> 51
- PU_EN1001: footprint project_fp:SolderJumper-2_Open_Pad0.5x1.0mm -> project_fp:SolderJumper-2_Open_Pad0.5x1.0mm_PU
Connections:
- net 3.3V_LDO: now also board_outline1.46, 3V3.2 (B); no longer T*C3.1, U2.5 (OUT)
- net 5V: now also board_outline1.45, 5V1.1 (A); no longer board_outline1.3 (Pin_3)
- net IOVDD: now also PU_EN1001.2; no longer PU_EN1001.1
- net at R1004.2, R1009.2: now also PU_EN1001.1; no longer PU_EN1001.2
- new net: 3V3.1 (A), T*C3.1, U2.5 (OUT)
- new net DSP_5V: 5V1.2 (B), board_outline1.3 (Pin_3)
Other:
- moved on the sheet: PU_EN1001

Commit message: update
Parts:
- added E1, E2, G1, G2: jumper, project_fp:jumper_slice, symbol proejct_lib:Jumper_2_Bridged
- added G10, G11, G3, G4, G5, G6, G7, G8, G9: VIA, project_fp:via, symbol proejct_lib:via
- 3V3: Label SC -> 3V
- 5V1: Label SC -> 5V
- ADD1001: footprint project_fp:SolderJumper-2_Open_Pad0.5x1.0mm -> project_fp:SolderJumper-2_Open_Pad0.5x1.0mm_ADDR; Label 50 -> 50 A0
- ADD1002: footprint project_fp:SolderJumper-2_Open_Pad0.5x1.0mm -> project_fp:SolderJumper-2_Open_Pad0.5x1.0mm_ADDR; Label 51 -> 51 A2
- ADD1003, ADD1004: footprint project_fp:SolderJumper-2_Open_Pad0.5x1.0mm -> project_fp:SolderJumper-2_Open_Pad0.5x1.0mm_ADDR
Connections:
- net Earth: now also D1007.2 (K), D1009.2 (K), E1.2 (B), E2.2 (B), G10.1, G11.1, G3.1, G4.1, G5.1, G6.1, G7.1, G8.1, G9.1; no longer board_outline1.E (AGND)
- net GNDD: now also G1.2 (B), G2.2 (B); no longer board_outline1.G (DGND)
- net 3.3V_A: now reaches 3V3.1 (A), T*C3.1, U2.5 (OUT)
- new net: G1.1 (A), board_outline1.49 (AGND)
- new net: E1.1 (A), board_outline1.47 (AGND)
- new net: E2.1 (A), board_outline1.48 (DGND)
- new net: G2.1 (A), board_outline1.50 (DGND)
Other:
- moved on the sheet: D1005
