File: tac5212_audio_board_single_ended.kicad_sch (KiCad schematic)
At the start: 94 parts, among them J1002 TAC5212, U1 Single Buffer - 74LVC1G125GV,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, U2 3.3v LDO - TLV74133PDQNR

Commit message: update
Parts:
- ADD1001: Label 50 A0 -> 50 A0
- ADD1002: Label 51 A2 -> 51 A2
- ADD1003: Label 52 A4 -> 52 A4
- ADD1004: Label 53 A6 -> 53 A6
- C1001: footprint V,+/- 10%, X7R, 0805 -> project_fp:C_0805_2012Metric
- OM1: footprint project_fp:jumper_slice_via -> project_fp:jumper_slice_via_alt_text
Connections:
- now unconnected: E1.1 (A), E2.1 (A), G1.1 (A), G2.1 (A), board_outline1.49 (AGND), board_outline1.50 (DGND)
Other:
- moved on the sheet: C1006, E1, E2, G1, G2

Commit message: update
Connections:
- net GNDD: no longer board_outline1.2 (Pin_2)
- net DSP_HELD_HIGH: no longer names the net of board_outline1.1 (HELD_HIGH)
- no-connect marks 0 -> 2
Changed lines of the file:
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@@
 		(color 0 0 0 0)
 	)
-	(junction
+	(no_connect
 		(at 257.81 271.78)
-		(diameter 0)
-		(color 0 0 0 0)
+	)
+	(no_connect
+		(at 208.28 271.78)
 	)
 	(wire
@@
 	(wire
 		(pts
-			(xy 257.81 271.78) (xy 265.43 271.78)
+			(xy 257.81 274.32) (xy 265.43 274.32)
 		)
 		(stroke
@@
 	(wire
 		(pts
-			(xy 196.85 340.36) (xy 208.28 340.36)
-		)
-		(stroke
-			(width 0)
-			(type default)
-		)
-	)
-	(wire
-		(pts
 			(xy 154.94 367.03) (xy 158.75 367.03)
 		)
@@
 	(wire
 		(pts
-			(xy 182.88 271.78) (xy 208.28 271.78)
-		)
-		(stroke
-			(width 0)
-			(type default)
-		)
-	)
-	(wire
-		(pts
 			(xy 66.04 123.19) (xy 66.04 116.84)
 		)
@@
 	(wire
 		(pts
-			(xy 257.81 271.78) (xy 257.81 274.32)
-		)
-		(stroke
-			(width 0)
-			(type default)
-		)
-	)
-	(wire
-		(pts
 			(xy 83.82 135.89) (xy 90.17 135.89)
 		)
@@
 		)
 	)
-	(label "DSP_HELD_HIGH"
-		(at 184.15 271.78 0)
-		(fields_autoplaced yes)
-		(effects
-			(font
-				(size 1.27 1.27)
-			)
-			(justify left bottom)
-		)
-	)
 	(label "GPI1"
 		(at 57.15 130.81 0)
@@
 	(global_label "3.3V_LDO"
 		(shape input)
-		(at 196.85 340.36 180)
+		(at 208.28 340.36 180)
 		(fields_autoplaced yes)
 		(effects
@@
 		)
 		(property "Intersheetrefs" "${INTERSHEET_REFS}"
-			(at 187.6426 340.36 0)
+			(at 199.0726 340.36 0)
 			(effects
 				(font
@@
 	(symbol
 		(lib_id "proejct_lib:GNDD")
-		(at 265.43 271.78 0)
+		(at 265.43 274.32 0)
 		(unit 1)
 		(exclude_from_sim no)
@@
 		(dnp no)
 		(property "Reference" "#PWR09"
-			(at 265.43 278.13 0)
+			(at 265.43 280.67 0)
 			(effects
 				(font
@@
 		)
 		(property "Value" "GNDD"
-			(at 265.43 287.782 0)
+			(at 265.43 290.322 0)
 			(effects
 				(font
@@
 		)
 		(property "Footprint" ""
-			(at 265.43 271.78 0)
+			(at 265.43 274.32 0)
 			(effects
 				(font
@@
 		)
 		(property "Datasheet" ""
-			(at 265.43 271.78 0)
+			(at 265.43 274.32 0)
 			(effects
 				(font
@@
 		)
 		(property "Description" ""
-			(at 265.43 271.78 0)
+			(at 265.43 274.32 0)
 			(effects
 				(font

Commit message: update
Parts:
- removed MK1001: SPH0611LR5H-1, SPH0611LR5H-1:XDCR_SPH0611LR5H-1, symbol proejct_lib:SPH0611LR5H-1
- 3V3, 5V1, E1, E2, G1, G2, GND1, MCLK1, SCL1001, SDA1001: PCBWAY_2020-06-09 NO COMPONENT -> (none); PCBWAY_2020-08-27 NO COMPONENT -> (none); PCBWAY_2020_04_18 NO COMPONENT -> (none)
- ADD1001, ADD1002, ADD1003, ADD1004, D1002, D1003, D1004, D1006, D1007, D1008, D1009, DOUT1, INM1, INM2, INP1, INP2, OM1, OM2, OP1, OP2, PU_EN1001: Part Number 2020-05-29 NO COMPONENT -> (none); Part Number 2020-08-26 NO COMPONENT -> (none); Part Number 2020-09-07 NO NEED TO PURCHASE OR MOUNT -> (none)
- C1: Manufacturer KEMET -> (none); Manufacturer_Part_Number C0805C104K5RAC7411 -> (none); mouser 80-C0805C104K5RACLR -> (none)
- C1010, C1011, C1013, C1014: 2024-01-06 UUQ1C100MCL1GB -> (none)
- C1012: SPEC CAP_100u_20%_25V_ALUM_RADIAL -> (none)
- C1015: Manufacturer Wurth Elektronik -> (none); Manufacturer_Part_Number 860020472006 -> (none); mouser 710-860020472006 -> (none)
- C1016, C1017, C1018, C1019, C1020: Digikey C1608X7R1H473K -> (none); Manufacturer TDK -> (none); Manufacturer_Part_Number C1608X7R1H473K080AA -> (none); mouser 810-C1608X7R1H473K -> (none)
- R1: mouser 603-RC0805DR-072K2L -> (none)
- R1001, R1002, R1003: Part Number 2020-05-29 ERJ-UP3J222V -> (none); Part Number 2020-08-26 ERJ-PA2F2211X (2.21k) -> (none); Part Number 2020-09-07 ERJ-PA2F2211X (2.21k) -> (none)
- R1016, R1018: Digikey ERJ-3EKF1000V -> (none); Manufacturer Bourns -> (none); Manufacturer_Part_Number CMP0805AFX-1000ELF -> (none); mouser 652-CMP0805AFX-1000L -> (none)
- R5: Digikey P100BYCT-ND -> (none); Manufacturer Bourns -> (none); Manufacturer_Part_Number CMP0805AFX-1000ELF -> (none); mouser 652-CMP0805AFX-1000L -> (none)
- T*C1, T*C3: Manufacturer Taiyo Yuden -> (none); Manufacturer_Part_Number LMR212BD7106KG-T -> (none); mouser 963-LMR212BD7106KG-T -> (none)
- T*C2: Manufacturer Kyocera AVX -> (none); Manufacturer_Part_Number 08055C104M4T4A -> (none); mouser 581-08055C104M4T4A -> (none)
- U1: Manufacturer TI / Nexperia -> (none); Manufacturer_Part_Number 74LVC1G125GV,125 -> (none); mouser 771-74LVC1G125GV -> (none)
- board_outline1: Digikey - -> (none); Manufacturer - -> (none); Manufacturer_Part_Number - -> (none); mouser - -> (none)
Connections:
- net at G1.1 (A): now also board_outline1.51 (DGND)
- net at board_outline1.49 (AGND): now also E1.1 (A)
- net at board_outline1.50 (AGND): now also E2.1 (A)
- net at board_outline1.52 (DGND): now also G2.1 (A)
- net DREG: no longer names the net of C1003.1, C1005.1, J1002.1 (DREG)
- net DSP_12V: no longer names the net of board_outline1.5 (12V)
- net DSP_5V: no longer names the net of 5V1.2 (B), board_outline1.3 (5V)
- no-connect marks 2 -> 3
Other:
- note added: "AUDIO FILTERS"
- note added: "DATA OUTPUT BUFFER"
- note added: "MODULE IO"
- note added: "POWER INDICATOR"
- note added: "POWER SUPPLY"
- note added: "TAC5212 AUDIO BREAKOUT MODULE"
- note added: "TAC5212 AUDIO CODEC"
- note removed: "DATA BUFFER"
- note removed: "POWER"
- note removed: "POWER SUPPLIES"
- note removed: "Suggested Sequence 1. IOVDD 2. AVDD, DRVDD 3. DVDD"
- note removed: "TAC5212 SINGLE ENDED"
- moved on the sheet: 3V3, 5V1, ADD1001, ADD1002, ADD1003, ADD1004, C1, C1001, C1002, C1003, C1004, C1005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

Commit message: update
Parts:
- added ADD1: jumper, project_fp:SolderJumper-2_Open_Pad0.5x1.0mm_ADDR, symbol proejct_lib:Jumper_NO_Small-Device
- 3V3, 5V1, ADD1001, ADD1002, ADD1003, ADD1004, DOUT1, E1, E2, G1, G10, G11, G2, G3, G4, G5, G6, G7, G8, G9, GND1, INM1, INM2, INP1, INP2, MCLK1, OM1, OM2, OP1, OP2, PU_EN1001, SCL1001, SDA1001: Package / Case (none) -> DNP; TAC5212EVM (none) -> n/a; now not fitted
- C1, T*C2: footprint project_fp:C_0805_2012Metric_Pad1.18x1.45mm_HandSolder -> Capacitor_SMD:C_0603_1608Metric_Pad1.08x0.95mm_HandSolder; Package / Case C0805 -> C0603; TAC5212EVM (none) -> C1608X7R1V105K080AC
- C1001: footprint project_fp:C_0805_2012Metric -> project_fp:C_0805_2012Metric_Pad1.18x1.45mm_HandSolder; Package / Case (none) -> C0805; TAC5212EVM (none) -> EMK212BB7106KG-T
- C1002, C1003: footprint Capacitor_SMD:C_0805_2012Metric -> project_fp:C_0805_2012Metric_Pad1.18x1.45mm_HandSolder; Package / Case (none) -> C0805; TAC5212EVM (none) -> EMK212BB7106KG-T
- C1004: footprint Capacitor_SMD:C_0603_1608Metric -> Capacitor_SMD:C_0603_1608Metric_Pad1.08x0.95mm_HandSolder; Package / Case (none) -> C0603; TAC5212EVM (none) -> C1608X7R1V105K080AC
- C1005, C1006, C1007: Package / Case (none) -> C0402; TAC5212EVM (none) -> GRM155R71C104KA88J
- C1008: Package / Case (none) -> C0603; TAC5212EVM (none) -> C1608X7R1V105K080AC
- C1009: value 0.1UF - 100V Ceramic Chip Capacitor, ±10%, X7R -> 10UF; EVM 16V Ceramic Chip Capacitor, ±10%, X7R -> (none); Package / Case C0805 -> C0603; TAC5212EVM (none) -> C1608X5R1C106M080AB
- C1010, C1011: value 0.1UF - 100V Ceramic Chip Capacitor, ±10%, X7R -> 10UF; Package / Case (none) -> C0603; TAC5212EVM (none) -> C1608X5R1C106M080AB
- C1012: value CAP CER 4.7UF 50V X7R 1206 - CAP ALUM 4.7UF 20% 50V RADIAL -> 10UF; TAC5212EVM (none) -> C1608X5R1C106M080AB
- C1013, C1014: value 47UF CAP CER 6.3V X5R 1210 - 47uF Radial -> 47uF; Package / Case (none) -> 3528-21; TAC5212EVM (none) -> TPSB476K010R0500
- C1015: value 47UF CAP CER 6.3V X5R 1210 - 47uF Radial -> 47uF; Package / Case through-5mm -> 3528-21; TAC5212EVM (none) -> TPSB476K010R0500
- C1016: value 47UF CAP CER 6.3V X5R 1210 - 47uF Radial -> 47uF; Package / Case C0805 -> 3528-21; TAC5212EVM (none) -> TPSB476K010R0500
- C1017, C1018, C1019, C1020: value 47NF CAP CER 100V X7R 0805 -> 0.047uF; footprint project_fp:C_0805_2012Metric_Pad1.18x1.45mm_HandSolder -> Capacitor_SMD:C_0603_1608Metric_Pad1.08x0.95mm_HandSolder; Package / Case C0805 -> C0603; TAC5212EVM (none) -> C1608X7R1H473K080AA
- D1002, D1003, D1004, D1005, D1006, D1007, D1008, D1009: Package / Case (none) -> D0402; TAC5212EVM (none) -> TPD1E10B06DPYR
- D7: value LED - B2601USD-20D000423U1930 -> RED LED; footprint project_fp:LED_1206_3216Metric_Pad1.42x1.75mm_HandSolder -> project_fp:R_0805_2012Metric_Pad1.20x1.40mm_HandSolder; Package / Case (none) -> 1206(CHECKME); TAC5212EVM (none) -> LTST-C170KRKT
- FB1001, FB1002, FB1003, FB1004: Package / Case (none) -> C0805; TAC5212EVM (none) -> BLM21A601S - BLM21AG601SH1
- J1002: Package / Case (none) -> 4X4; TAC5212EVM (none) -> TAC5212
- R1: footprint project_fp:R_0805_2012Metric_Pad1.20x1.40mm_HandSolder -> Resistor_SMD:R_0402_1005Metric_Pad0.72x0.64mm_HandSolder; TAC5212EVM (none) -> RC0402FR-7W49R9L
- R1001, R1003: value 4.7KOhm -> 4.7k; Package / Case (none) -> R0402; TAC5212EVM (none) -> ERJ-3GEYJ472V
- R1002: value 22KOhm -> 22.0k; Package / Case (none) -> R0402; TAC5212EVM (none) -> RG1608P-223-B-T5
- R1004, R1009: Package / Case (none) -> R0402; TAC5212EVM (none) -> RC0402FR-07100KL
- R1005, R1006, R1007, R1008, R1010, R1011, R1012, R1013: Package / Case (none) -> R0402; TAC5212EVM (none) -> ERJ-2GE0R00X
- R1015: value 100ohm -> 100; footprint project_fp:R_0805_2012Metric_Pad1.20x1.40mm_HandSolder -> project_fp:R_0603_1608Metric_Pad1.05x0.95mm_HandSolder; Package / Case (none) -> R0603; TAC5212EVM (none) -> RC0603FR-07100RL
- R1016: value 1K RES SMD OHM 1% 1/2W 0805 -> 100; footprint project_fp:R_0805_2012Metric_Pad1.20x1.40mm_HandSolder -> project_fp:R_0603_1608Metric_Pad1.05x0.95mm_HandSolder; Package / Case R0805 -> R0603; TAC5212EVM (none) -> RC0603FR-07100RL
- R1017: value 1K RES SMD OHM 1% 1/2W 0805 -> 100; footprint project_fp:R_0805_2012Metric_Pad1.20x1.40mm_HandSolder -> project_fp:R_0603_1608Metric_Pad1.05x0.95mm_HandSolder; Package / Case (none) -> R0603; TAC5212EVM (none) -> RC0603FR-07100RL
- R1018: value 100ohm -> 100; footprint project_fp:R_0805_2012Metric_Pad1.20x1.40mm_HandSolder -> project_fp:R_0603_1608Metric_Pad1.05x0.95mm_HandSolder; Package / Case R0805 -> R0603; TAC5212EVM (none) -> RC0603FR-07100RL
- R5: footprint project_fp:R_0805_2012Metric_Pad1.20x1.40mm_HandSolder -> Resistor_SMD:R_0402_1005Metric; Package / Case R0805 -> R0402; TAC5212EVM (none) -> RC0402FR-07100KL
- T*C1, T*C3: value DNP (10uF) -> 10uF; TAC5212EVM (none) -> EMK212BB7106KG-T
- U1: Package / Case SC70-5 -> SOT-23-5; TAC5212EVM (none) -> 74LVC1G125GV,125
- U2: value 3.3v LDO - TLV74133PDQNR -> 3.3v LDO - TLV74133PDBVR; Package / Case (none) -> SOT-23-5; TAC5212EVM (none) -> TLV74133PDBVR
- board_outline1: Package / Case board -> DNP; TAC5212EVM (none) -> n/a
Connections:
- net 3.3V_LDO: now also ADD1.2
- net at ADD1001.2, ADD1002.2, ADD1003.2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: now also ADD1.1
Other:
- moved on the sheet: R1001, R1002, R1003
