File: tac5212_audio_board_single_ended.kicad_sch (KiCad schematic)
At the start: 106 parts, among them T108 Tab, T109 Tab, T110 Tab, T111 Tab, U108 Single Buffer with Tri-state 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, U109 3.3v LDO - TLV74133PDBVR

Commit message: update
Parts:
- added G120, G121, G122, G124, INM1, INM2, INP1, INP2, OUTM1, OUTM2, OUTP1, OUTP2: VIA, project_fp:via, symbol proejct_lib:via
- added G123: SMD ROUTING PAD, project_fp:SMD_ROUTING_PAD, symbol proejct_lib:via
Connections:
- net Earth: now also G120.1, G121.1, G122.1, G123.1
- net IN1M: now also INM1.1
- net IN1P: now also INP1.1
- net IN2M: now also INM2.1
- net IN2P: now also INP2.1
- net OUT1M: now also R109.2, R111.2, OUTM1.1
- net OUT1M+: now also C117.2, D109.1 (K), R116.1; no longer C110.2, D108.1 (K), R129.1
- net OUT1P: now also OUTP1.1; no longer R109.2, R111.2, R131.2, R132.2, R134.2, R135.2
- net OUT1P+: now also C110.2, D108.1 (K), R129.1; no longer C117.2, D109.1 (K), R116.1
- net OUT2M: now also R134.2, R135.2, OUTM2.1
- net OUT2P: now also R131.2, R132.2, OUTP2.1
Other:
- moved on the sheet: G108, G109, G110, G111, G112

Commit message: update
Parts:
- C129: value 1uF is this the right value? -> 0.1uF; footprint project_fp:C_0603_1608Metric_Pad1.08x0.95mm_HandSolder -> project_fp:C_0402_1005Metric; Package / Case C0603 -> C0402; TAC5212EVM C1608X7R1V105K080AC -> GRM155R71C104KA88J
- FB108, FB109, FB110, FB111: footprint project_fp:C_0805_2012Metric_Pad1.18x1.45mm_HandSolder_alt_location -> project_fp:C_0805_2012Metric_Pad1.18x1.45mm_HandSolder
- G108, G109, G110, G111, G112: footprint project_fp:via -> project_fp:SMD_ROUTING_PAD
- R128: now not fitted
Changed lines of the file:
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@@
 			)
 		)
-		(property "Footprint" "project_fp:C_0805_2012Metric_Pad1.18x1.45mm_HandSolder_alt_location"
+		(property "Footprint" "project_fp:C_0805_2012Metric_Pad1.18x1.45mm_HandSolder"
 			(at 520.7 295.148 90)
 			(effects
@@
 			)
 		)
-		(property "Footprint" "project_fp:C_0805_2012Metric_Pad1.18x1.45mm_HandSolder_alt_location"
+		(property "Footprint" "project_fp:C_0805_2012Metric_Pad1.18x1.45mm_HandSolder"
 			(at 513.08 376.428 90)
 			(effects
@@
 			)
 		)
-		(property "Footprint" "project_fp:C_0805_2012Metric_Pad1.18x1.45mm_HandSolder_alt_location"
+		(property "Footprint" "project_fp:C_0805_2012Metric_Pad1.18x1.45mm_HandSolder"
 			(at 516.89 417.068 90)
 			(effects
@@
 			)
 		)
-		(property "Footprint" "project_fp:via"
+		(property "Footprint" "project_fp:SMD_ROUTING_PAD"
 			(at 368.3 217.17 0)
 			(effects
@@
 			)
 		)
-		(property "Footprint" "project_fp:via"
+		(property "Footprint" "project_fp:SMD_ROUTING_PAD"
 			(at 368.3 115.57 0)
 			(effects
@@
 		(exclude_from_sim no)
 		(in_bom no)
-		(on_board yes)
+		(on_board no)
 		(dnp yes)
 		(property "Reference" "SCL109"
@@
 			)
 		)
-		(property "Footprint" "project_fp:via"
+		(property "Footprint" "project_fp:SMD_ROUTING_PAD"
 			(at 368.3 182.88 0)
 			(effects
@@
 		(exclude_from_sim no)
 		(in_bom yes)
-		(on_board yes)
-		(dnp no)
+		(on_board no)
+		(dnp yes)
 		(property "Reference" "R128"
 			(at 61.722 343.408 90)
@@
 			)
 		)
-		(property "Footprint" "project_fp:C_0805_2012Metric_Pad1.18x1.45mm_HandSolder_alt_location"
+		(property "Footprint" "project_fp:C_0805_2012Metric_Pad1.18x1.45mm_HandSolder"
 			(at 515.62 329.438 90)
 			(effects
@@
 			)
 		)
-		(property "Footprint" "project_fp:via"
+		(property "Footprint" "project_fp:SMD_ROUTING_PAD"
 			(at 370.84 92.71 0)
 			(effects
@@
 			)
 		)
-		(property "Footprint" "project_fp:via"
+		(property "Footprint" "project_fp:SMD_ROUTING_PAD"
 			(at 368.3 148.59 0)
 			(effects
@@
 			)
 		)
-		(property "Value" "1uF is this the right value?"
+		(property "Value" "0.1uF"
 			(at 65.8368 346.583 0)
 			(effects
@@
 			)
 		)
-		(property "Footprint" "project_fp:C_0603_1608Metric_Pad1.08x0.95mm_HandSolder"
+		(property "Footprint" "project_fp:C_0402_1005Metric"
 			(at 63.5 345.44 0)
 			(effects
@@
 			)
 		)
-		(property "Description" "CAP, CERM, 1 uF, 35 V, +/- 10%, X7R, 0603"
+		(property "Description" "CAP, CERM, 0.1 uF, 16 V, +/- 10%, X7R, 0402"
 			(at 63.5 345.44 0)
 			(effects
@@
 			)
 		)
-		(property "Package / Case" "C0603"
+		(property "Package / Case" "C0402"
 			(at 63.5 345.44 0)
 			(effects
@@
 			)
 		)
-		(property "TAC5212EVM" "C1608X7R1V105K080AC"
+		(property "TAC5212EVM" "GRM155R71C104KA88J"
 			(at 63.5 345.44 0)
 			(effects
