File: t-dsp_tac5212_pro_audio_module.kicad_sch (KiCad schematic)
At the start: 119 parts, among them T108 Tab, T109 Tab, T110 Tab, T111 Tab, U108 Single Buffer with Tri-state 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, U109 3.3v LDO - TLV74133PDBVR

Commit message: Rename project to T-DSP TAC5212 Pro Audio Module
- Rename all KiCad project files from tac5212_audio_board_single_ended
  to t-dsp_tac5212_pro_audio_module
- Update internal filename references in .kicad_pro and .kicad_prl
- Rename schematic/footprint PDFs and move to documentation/
- Update README: new title, corrected connector/module descriptions,
  add 3D renders, pinout diagram, interactive BOM link, and docs links
- Update kikit_script.txt with new project filenames
- Clean up .gitignore (remove redundant lock file entry)
- Add LICENSE (CC BY-NC-SA 4.0)

Co-Authored-By: Claude Opus 4.6 <noreply@anthropic.com>
Other:
- note added: "T-DSP TAC5212 Pro Audio Module"
- note removed: "TAC5212 AUDIO BREAKOUT MODULE"
Changed lines of the file:
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@@
 		)
 	)
-	(text "TAC5212 AUDIO BREAKOUT MODULE"
+	(text "T-DSP TAC5212 Pro Audio Module"
 		(exclude_from_sim no)
 		(at 39.37 37.084 0)
