File: t-dsp_tac5212_pro_audio_module.kicad_sch (KiCad schematic)
At the start: 119 parts, among them J3V108 jumper, J5V108 jumper, T108 Tab, T109 Tab, T110 Tab, T111 Tab, U108 Single Buffer with Tri-state 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, U109 3.3v LDO - TLV74133PDBVR

Commit message: Add LCSC part number for U108 (SN74LVC1G66DCK)
Add C113518 to complete JLCPCB BOM coverage for all active components.
Parts:
- U108: LCSC (none) -> C113518
Changed lines of the file:
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@@
+			)
+		)
+		(property "LCSC" "C113518"
+			(at 185.42 284.48 0)
+			(effects
+				(font
+					(size 1.27 1.27)
+				)
+				(hide yes)
 			)
 		)

Commit message: Add LCSC enrichment, iBOM, and consolidate manufacturing pipeline
- Enrich schematic with LCSC_Manufacturer and LCSC_MPN for all components
- Add enrichment and verification scripts (scripts/)
- Consolidate all outputs into single project-named folder
- Both BOMs (JLCPCB + generic with MPN) included in manufacturing ZIP
- Add interactive BOM generation and GitHub Pages deployment
- Remove deprecated gerber/, bom/, and panel/ folders (replaced by CI)
Parts:
- C108, C111, C115, C131, T*C108, T*C110: LCSC_MPN (none) -> EMK212BB7106KG-T; LCSC_Manufacturer (none) -> Taiyo Yuden
- C109, C112, C116, C128, C129: LCSC_MPN (none) -> GRM155R71C104KA88J; LCSC_Manufacturer (none) -> muRata
- C110, C117, C121, C123: LCSC_MPN (none) -> TPSB476K010R0500; LCSC_Manufacturer (none) -> Kyocera AVX
- C113, C114, C120, C122: LCSC_MPN (none) -> C1608X7R1H473K080AA; LCSC_Manufacturer (none) -> TDK
- C118, C119, T*C109: LCSC_MPN (none) -> C1608X7R1V105K080AC; LCSC_Manufacturer (none) -> TDK
- C124, C125, C126, C127: LCSC_MPN (none) -> C1608X5R1C106M080AB; LCSC_Manufacturer (none) -> TDK
- C130: LCSC_MPN (none) -> CL21A476MQYNNNE; LCSC_Manufacturer (none) -> Samsung Electro-Mechanics
- D108, D109, D110, D111, D112, D113, D114, D115: LCSC_MPN (none) -> TPD1E10B06DPYR; LCSC_Manufacturer (none) -> TI
- D116: LCSC_MPN (none) -> LTST-C170KRKT; LCSC_Manufacturer (none) -> LITEON
- FB108, FB109, FB110, FB111: LCSC_MPN (none) -> BLM21AG601SH1D; LCSC_Manufacturer (none) -> muRata
- R108, R111, R132, R135: LCSC_MPN (none) -> 0603WAF100JT5E; LCSC_Manufacturer (none) -> UNI-ROYAL
- R115, R118, R119: LCSC_MPN (none) -> ERJ2GE0R00X; LCSC_Manufacturer (none) -> PANASONIC
- R116, R129, R133, R136: LCSC_MPN (none) -> 0603WAF0000T5E; LCSC_Manufacturer (none) -> UNI-ROYAL
- R117, R125: LCSC_MPN (none) -> 0402WGF330JTCE; LCSC_Manufacturer (none) -> UNI-ROYAL
- R120, R121, R128: LCSC_MPN (none) -> RC0402FR-072K21L; LCSC_Manufacturer (none) -> YAGEO
- R122: LCSC_MPN (none) -> RC0402FR-0722KL; LCSC_Manufacturer (none) -> YAGEO
- R123, R124: LCSC_MPN (none) -> ERJ3GEYJ472V; LCSC_Manufacturer (none) -> PANASONIC
- R126: LCSC_MPN (none) -> RC0402FR-07100KL; LCSC_Manufacturer (none) -> YAGEO
- R130, R137, R138, R139: LCSC_MPN (none) -> 0603WAF1003T5E; LCSC_Manufacturer (none) -> UNI-ROYAL
- TAC5212: LCSC_MPN (none) -> TAC5212IRGER; LCSC_Manufacturer (none) -> TI
- U108: LCSC_MPN (none) -> SN74LVC1G66DCKR; LCSC_Manufacturer (none) -> TI
- U109: LCSC_MPN (none) -> TLV74133PDBVR; LCSC_Manufacturer (none) -> TI
