File: t-dsp_tac5212_pro_audio_module.kicad_sch (KiCad schematic)
At the start: 119 parts, among them J3V108 jumper, J5V108 jumper, T108 Tab, T109 Tab, T110 Tab, T111 Tab, U108 Single Buffer with Tri-state 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, U109 3.3v LDO - TLV74133PDBVR

Commit message: Fix BOM field conflicts and component data errors
- Fix R126 LCSC code (C60491 100K -> C138019 2.21K) in schematic and PCB
- Fix Package/Case mismatches in PCB: C128 (C0603->C0402), C124 (C0805->C0603)
- Fix Description fields: remove MISMATCH FOOTPRINT notes, correct 0603->0402
  for R122, R123, R124; unify R125 description to match R117
- Fix D116 LED Package/Case from 1206(CHECKME) to 0805
- Add schematic PDF and PCB layout PDF to manufacturing ZIP

Co-Authored-By: Claude Opus 4.6 <noreply@anthropic.com>
Parts:
- D116: Package / Case 1206(CHECKME) -> 0805
- R126: LCSC C60491 -> C138019; LCSC_MPN RC0402FR-07100KL -> RC0402FR-072K21L; REPLACE FOR NEXT BUILD RC0402FR-072K21L -> (none); TAC5212EVM RC0402FR-07100KL -> RC0402FR-072K21L
Changed lines of the file:
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@@
 			)
 		)
-		(property "Package / Case" "1206(CHECKME)"
+		(property "Package / Case" "0805"
 			(at 139.7 529.59 0)
 			(effects
@@
 			)
 		)
-		(property "Description" "MISMATCH FOOTPRINT  RES, 22.0 k, 0.1%, 0.1 W, 0603"
+		(property "Description" "RES, 22.0 k, 0.1%, 0.1 W, 0402"
 			(at 91.44 168.91 0)
 			(effects
@@
 			)
 		)
-		(property "TAC5212EVM" "RC0402FR-07100KL"
+		(property "TAC5212EVM" "RC0402FR-072K21L"
 			(at 130.81 528.32 0)
 			(effects
@@
 			)
 		)
-		(property "REPLACE FOR NEXT BUILD" "RC0402FR-072K21L"
+		(property "REPLACE FOR NEXT BUILD" ""
 			(at 130.81 528.32 0)
 			(effects
@@
 			)
 		)
-		(property "LCSC" "C60491"
+		(property "LCSC" "C138019"
 			(at 130.81 528.32 0)
 			(effects
@@
 			)
 		)
-		(property "LCSC_MPN" "RC0402FR-07100KL"
+		(property "LCSC_MPN" "RC0402FR-072K21L"
 			(at -69.85 179.07 0)
 			(effects
@@
 			)
 		)
-		(property "Description" "RES 27 ohm 1% 1/8W 0402"
+		(property "Description" "RES SMD 27 ohm 1/10W 0402"
 			(at 146.05 450.85 0)
 			(effects
@@
 			)
 		)
-		(property "Description" "MISMATCH FOOTPRINT -RES, 4.7 k, 5%, 0.1 W, AEC-Q200 Grade 0, 0603"
+		(property "Description" "RES, 4.7 k, 5%, 0.1 W, 0402"
 			(at 91.44 177.8 0)
 			(effects
@@
 			)
 		)
-		(property "Description" "MISMATCH FOOTPRINT -RES, 4.7 k, 5%, 0.1 W, AEC-Q200 Grade 0, 0603"
+		(property "Description" "RES, 4.7 k, 5%, 0.1 W, 0402"
 			(at 91.44 200.66 0)
 			(effects
