File: panel/jlcpcb_4x4/jlcpcb_4x4.kicad_pcb (KiCad board)
At the start: 4 copper layers, 70.5 x 100 mm, 532 parts, among them U108 Single Buffer - 74LVC1G125GV,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, U109 3.3v LDO - TLV74133PDBVR

Commit message: fab
Parts:
- removed the 3V108 at (138.7, 34.8)
- removed the 3V108 at (138.7, 78.8)
- removed the 3V108 at (167.2, 34.8)
- removed the 3V108 at (167.2, 78.8)
- removed the 5V108 at (144.4, 60.9)
- removed the 5V108 at (172.9, 104.9)
- removed the 5V108 at (172.9, 60.9)
- removed the 5V108 at (144.4, 104.9)
- removed the ADD108 at (134.0, 36.8)
- removed the ADD108 at (162.5, 36.8)
- removed the ADD108 at (134.0, 80.8)
- removed the ADD108 at (162.5, 80.8)
- removed the ADD110 at (134.0, 33.6)
- removed the ADD110 at (134.0, 77.6)
- removed the ADD110 at (162.5, 33.6)
- removed the ADD110 at (162.5, 77.6)
- removed the ADD111 at (162.5, 32.0)
- removed the ADD111 at (134.0, 32.0)
- removed the ADD111 at (134.0, 76.0)
- removed the ADD111 at (162.5, 76.0)
- removed the ADD112 at (134.0, 35.2)
- removed the ADD112 at (134.0, 79.2)
- removed the ADD112 at (162.5, 35.2)
- removed the ADD112 at (162.5, 79.2)
- removed the C108 at (133.0, 51.8)
- removed the C108 at (161.5, 51.8)
- removed the C108 at (161.5, 95.8)
- removed the C108 at (133.0, 95.8)
- removed the C109 at (160.4, 48.6)
- removed the C109 at (131.9, 48.6)
- removed the C109 at (160.4, 92.6)
- removed the C109 at (131.9, 92.6)
- removed the C110 at (166.5, 100.5)
- removed the C110 at (166.5, 56.5)
- removed the C110 at (138.0, 100.5)
- removed the C110 at (138.0, 56.5)
- removed the C111 at (141.3, 92.8)
- removed the C111 at (141.3, 48.8)
- removed the C111 at (169.8, 48.8)
- removed the C111 at (169.8, 92.8)
- removed the C112 at (168.2, 45.6)
- removed the C112 at (139.7, 45.6)
- removed the C112 at (168.2, 89.6)
- removed the C112 at (139.7, 89.6)
- removed the C113 at (159.6, 100.1)
- removed the C113 at (159.6, 56.1)
- removed the C113 at (131.1, 100.1)
- removed the C113 at (131.1, 56.1)
- removed the C114 at (138.0, 60.8)
- removed the C114 at (166.5, 60.8)
- removed the C114 at (138.0, 104.8)
- removed the C114 at (166.5, 104.8)
- removed the C115 at (136.8, 52.4)
- removed the C115 at (165.3, 96.4)
- removed the C115 at (165.3, 52.4)
- removed the C115 at (136.8, 96.4)
- removed the C116 at (135.7, 49.4)
- removed the C116 at (135.7, 93.4)
- removed the C116 at (164.2, 93.4)
- removed the C116 at (164.2, 49.4)
- removed the C117 at (131.1, 60.4)
- removed the C117 at (159.6, 104.4)
- removed the C117 at (131.1, 104.4)
- removed the C117 at (159.6, 60.4)
- removed the C118 at (155.8, 73.6)
- removed the C118 at (155.8, 29.6)
- removed the C118 at (127.3, 73.6)
- removed the C118 at (127.3, 29.6)
- removed the C119 at (163.0, 94.6)
- removed the C119 at (134.5, 50.6)
- removed the C119 at (163.0, 50.6)
- removed the C119 at (134.5, 94.6)
- removed the C120 at (166.5, 52.2)
- removed the C120 at (166.5, 96.2)
- removed the C120 at (138.0, 96.2)
- removed the C120 at (138.0, 52.2)
- removed the C121 at (159.6, 95.8)
- removed the C121 at (131.1, 51.8)
- removed the C121 at (131.1, 95.8)
- removed the C121 at (159.6, 51.8)
- removed the C122 at (138.9, 47.1)
- removed the C122 at (167.4, 91.1)
- removed the C122 at (138.9, 91.1)
- removed the C122 at (167.4, 47.1)
- removed the C123 at (159.6, 91.9)
- removed the C123 at (131.1, 91.9)
- removed the C123 at (159.6, 47.9)
- removed the C123 at (131.1, 47.9)
- removed the C124 at (163.0, 75.0)
- removed the C124 at (134.5, 31.0)
- removed the C124 at (163.0, 31.0)
- removed the C124 at (134.5, 75.0)
- removed the C125 at (163.1, 33.6)
- removed the C125 at (134.6, 77.6)
- removed the C125 at (163.1, 77.6)
- removed the C125 at (134.6, 33.6)
- removed the C126 at (134.5, 81.2)
- removed the C126 at (163.0, 37.2)
- removed the C126 at (163.0, 81.2)
- removed the C126 at (134.5, 37.2)
- removed the C127 at (134.5, 39.9)
- removed the C127 at (134.5, 83.9)
- removed the C127 at (163.0, 39.9)
- removed the C127 at (163.0, 83.9)
- removed the C128 at (141.1, 57.0)
- removed the C128 at (169.6, 57.0)
- removed the C128 at (169.6, 101.0)
- removed the C128 at (141.1, 101.0)
- removed the C129 at (139.9, 41.5)
- removed the C129 at (168.3, 85.5)
- removed the C129 at (139.9, 85.5)
- removed the C129 at (168.3, 41.5)
- removed the C130 at (171.0, 104.6)
- removed the C130 at (142.5, 104.6)
- removed the C130 at (171.0, 60.6)
- removed the C130 at (142.5, 60.6)
- removed the C131 at (144.7, 104.6)
- removed the C131 at (144.7, 60.6)
- removed the C131 at (173.2, 60.6)
- removed the C131 at (173.2, 104.6)
- removed the D108 at (128.2, 100.9)
- removed the D108 at (128.2, 56.9)
- removed the D108 at (156.7, 100.9)
- removed the D108 at (156.7, 56.9)
- removed the D109 at (128.2, 61.2)
- removed the D109 at (128.2, 105.2)
- removed the D109 at (156.7, 61.2)
- removed the D109 at (156.7, 105.2)
- removed the D110 at (156.7, 52.6)
- removed the D110 at (128.2, 96.6)
- removed the D110 at (156.7, 96.6)
- removed the D110 at (128.2, 52.6)
- removed the D111 at (128.2, 92.9)
- removed the D111 at (128.2, 48.9)
- removed the D111 at (156.7, 92.9)
- removed the D111 at (156.7, 48.9)
- removed the D112 at (156.6, 74.2)
- removed the D112 at (128.2, 74.2)
- removed the D112 at (128.2, 30.2)
- removed the D112 at (156.6, 30.2)
- removed the D113 at (156.6, 33.8)
- removed the D113 at (156.6, 77.8)
- removed the D113 at (128.1, 33.8)
- removed the D113 at (128.1, 77.8)
- removed the D114 at (156.6, 37.4)
- removed the D114 at (128.1, 37.4)
- removed the D114 at (156.6, 81.4)
- removed the D114 at (128.1, 81.4)
- removed the D115 at (156.5, 85.0)
- removed the D115 at (128.0, 41.0)
- removed the D115 at (128.0, 85.0)
- removed the D115 at (156.5, 41.0)
- removed the D116 at (140.2, 33.6)
- removed the D116 at (168.7, 33.6)
- removed the D116 at (140.2, 77.6)
- removed the D116 at (168.7, 77.6)
- removed the DOUT108 at (138.5, 54.5)
- removed the DOUT108 at (138.5, 98.5)
- removed the DOUT108 at (167.0, 54.5)
- removed the DOUT108 at (167.0, 98.5)
- removed the E108 at (122.8, 98.1)
- removed the E108 at (151.3, 54.1)
- removed the E108 at (151.3, 98.1)
- removed the E108 at (122.8, 54.1)
- removed the E109 at (151.3, 75.7)
- removed the E109 at (151.3, 31.7)
- removed the E109 at (122.8, 31.7)
- removed the E109 at (122.8, 75.7)
- removed the FB108 at (159.3, 30.3)
- removed the FB108 at (159.3, 74.3)
- removed the FB108 at (130.9, 30.3)
- removed the FB108 at (130.9, 74.3)
- removed the FB109 at (130.8, 77.9)
- removed the FB109 at (159.3, 33.9)
- removed the FB109 at (159.3, 77.9)
- removed the FB109 at (130.8, 33.9)
- removed the FB110 at (130.8, 37.5)
- removed the FB110 at (130.8, 81.5)
- removed the FB110 at (159.2, 81.5)
- removed the FB110 at (159.2, 37.5)
- removed the FB111 at (159.1, 41.1)
- removed the FB111 at (130.6, 41.1)
- removed the FB111 at (130.6, 85.1)
- removed the FB111 at (159.1, 85.1)
- removed the G108 at (137.6, 38.0)
- removed the G108 at (137.6, 82.0)
- removed the G108 at (166.1, 82.0)
- removed the G108 at (166.1, 38.0)
- removed the G109 at (140.3, 98.6)
- removed the G109 at (168.8, 54.6)
- removed the G109 at (168.8, 98.6)
- removed the G109 at (140.3, 54.6)
- removed the G110 at (137.1, 80.7)
- removed the G110 at (137.1, 36.7)
- removed the G110 at (165.6, 36.7)
- removed the G110 at (165.6, 80.7)
- removed the G111 at (141.3, 61.8)
- removed the G111 at (169.8, 61.8)
- removed the G111 at (141.3, 105.8)
- removed the G111 at (169.8, 105.8)
- removed the G112 at (165.6, 79.4)
- removed the G112 at (137.1, 35.4)
- removed the G112 at (165.6, 35.4)
- removed the G112 at (137.1, 79.4)
- removed the G113 at (141.5, 51.6)
- removed the G113 at (170.0, 51.6)
- removed the G113 at (170.0, 95.6)
- removed the G113 at (141.5, 95.6)
- removed the G114 at (138.7, 74.8)
- removed the G114 at (167.2, 30.8)
- removed the G114 at (167.2, 74.8)
- removed the G114 at (138.7, 30.8)
- removed the G115 at (171.4, 92.8)
- removed the G115 at (171.4, 48.8)
- removed the G115 at (142.9, 92.8)
- removed the G115 at (142.9, 48.8)
- removed the G116 at (133.3, 71.9)
- removed the G116 at (133.3, 27.9)
- removed the G116 at (161.8, 71.9)
- removed the G116 at (161.8, 27.9)
- removed the G117 at (145.1, 98.3)
- removed the G117 at (145.1, 54.3)
- removed the G117 at (173.6, 54.3)
- removed the G117 at (173.6, 98.3)
- removed the G118 at (145.7, 75.6)
- removed the G118 at (145.7, 31.6)
- removed the G118 at (174.2, 31.6)
- removed the G118 at (174.2, 75.6)
- removed the G119 at (138.7, 76.2)
- removed the G119 at (167.2, 32.2)
- removed the G119 at (138.7, 32.2)
- removed the G119 at (167.2, 76.2)
- removed the GND108 at (156.6, 88.6)
- removed the GND108 at (128.1, 44.6)
- removed the GND108 at (128.1, 88.6)
- removed the GND108 at (156.6, 44.6)
- removed the INM1 at (130.0, 36.0)
- removed the INM1 at (158.4, 80.0)
- removed the INM1 at (130.0, 80.0)
- removed the INM1 at (158.4, 36.0)
- removed the INM2 at (158.5, 28.8)
- removed the INM2 at (130.1, 28.8)
- removed the INM2 at (158.5, 72.8)
- removed the INM2 at (130.1, 72.8)
- removed the INP1 at (130.0, 83.6)
- removed the INP1 at (158.5, 83.6)
- removed the INP1 at (158.5, 39.6)
- removed the INP1 at (130.0, 39.6)
- removed the INP2 at (130.0, 76.4)
- removed the INP2 at (158.5, 32.4)
- removed the INP2 at (130.0, 32.4)
- removed the INP2 at (158.5, 76.4)
- removed KiKit_MB_10_1, KiKit_MB_10_6, KiKit_MB_11_1, KiKit_MB_11_6, KiKit_MB_12_1, KiKit_MB_12_6, KiKit_MB_13_6, KiKit_MB_13_7, KiKit_MB_14_6, KiKit_MB_14_7, KiKit_MB_15_6, KiKit_MB_15_7, KiKit_MB_16_6, KiKit_MB_16_7, KiKit_MB_17_8, KiKit_MB_18_8, KiKit_MB_19_8, KiKit_MB_1_1, KiKit_MB_1_6, KiKit_MB_20_8, KiKit_MB_2_1, KiKit_MB_2_6, KiKit_MB_3_1, KiKit_MB_3_6, KiKit_MB_4_1, KiKit_MB_4_6, KiKit_MB_5_1, KiKit_MB_5_6, KiKit_MB_6_1, KiKit_MB_6_6, KiKit_MB_7_1, KiKit_MB_7_6, KiKit_MB_8_1, KiKit_MB_8_6, KiKit_MB_9_1, KiKit_MB_9_6: NPTH, NPTH
- removed the MCLK108 at (122.5, 61.0)
- removed the MCLK108 at (151.0, 61.0)
- removed the MCLK108 at (122.5, 105.0)
- removed the MCLK108 at (151.0, 105.0)
- removed the NT108 at (170.4, 30.2)
- removed the NT108 at (141.9, 30.2)
- removed the NT108 at (141.9, 74.2)
- removed the NT108 at (170.4, 74.2)
- removed the NT109 at (161.2, 49.2)
- removed the NT109 at (161.2, 93.2)
- removed the NT109 at (132.7, 93.2)
- removed the NT109 at (132.7, 49.2)
- removed the OM1 at (130.1, 61.8)
- removed the OM1 at (158.6, 105.8)
- removed the OM1 at (130.1, 105.8)
- removed the OM1 at (158.6, 61.8)
- removed the OM2 at (129.8, 49.6)
- removed the OM2 at (129.8, 93.6)
- removed the OM2 at (158.3, 49.6)
- removed the OM2 at (158.3, 93.6)
- removed the OP1 at (130.1, 57.8)
- removed the OP1 at (158.6, 101.8)
- removed the OP1 at (158.6, 57.8)
- removed the OP1 at (130.1, 101.8)
- removed the OP2 at (130.0, 97.5)
- removed the OP2 at (158.5, 97.5)
- removed the OP2 at (130.0, 53.5)
- removed the OP2 at (158.5, 53.5)
- removed the PU_EN108 at (141.7, 45.6)
- removed the PU_EN108 at (170.2, 45.6)
- removed the PU_EN108 at (141.7, 89.6)
- removed the PU_EN108 at (170.2, 89.6)
- removed the R108 at (162.7, 56.1)
- removed the R108 at (134.2, 100.1)
- removed the R108 at (134.2, 56.1)
- removed the R108 at (162.7, 100.1)
- removed the R109 at (134.2, 60.4)
- removed the R109 at (162.7, 104.4)
- removed the R109 at (162.7, 60.4)
- removed the R109 at (134.2, 104.4)
- removed the R110 at (164.4, 38.6)
- removed the R110 at (135.9, 82.6)
- removed the R110 at (164.4, 82.6)
- removed the R110 at (135.9, 38.6)
- removed the R111 at (162.7, 95.8)
- removed the R111 at (134.2, 95.8)
- removed the R111 at (134.2, 51.8)
- removed the R111 at (162.7, 51.8)
- removed the R112 at (165.2, 39.4)
- removed the R112 at (136.7, 39.4)
- removed the R112 at (165.2, 83.4)
- removed the R112 at (136.7, 83.4)
- removed the R113 at (166.0, 40.2)
- removed the R113 at (137.5, 84.2)
- removed the R113 at (137.5, 40.2)
- removed the R113 at (166.0, 84.2)
- removed the R114 at (138.3, 85.0)
- removed the R114 at (166.8, 41.0)
- removed the R114 at (166.8, 85.0)
- removed the R114 at (138.3, 41.0)
- removed the R115 at (165.8, 92.0)
- removed the R115 at (137.4, 92.0)
- removed the R115 at (137.4, 48.0)
- removed the R115 at (165.8, 48.0)
- removed the R116 at (163.6, 92.3)
- removed the R116 at (135.1, 48.3)
- removed the R116 at (135.1, 92.3)
- removed the R116 at (163.6, 48.3)
- removed the R117 at (166.5, 47.3)
- removed the R117 at (138.1, 47.3)
- removed the R117 at (166.5, 91.3)
- removed the R117 at (138.1, 91.3)
- removed the R118 at (167.2, 46.6)
- removed the R118 at (138.7, 46.6)
- removed the R118 at (167.2, 90.6)
- removed the R118 at (138.7, 90.6)
- removed the R119 at (165.2, 92.6)
- removed the R119 at (165.2, 48.6)
- removed the R119 at (136.7, 92.6)
- removed the R119 at (136.7, 48.6)
- removed the R120 at (139.7, 42.6)
- removed the R120 at (168.2, 42.6)
- removed the R120 at (139.7, 86.6)
- removed the R120 at (168.2, 86.6)
- removed the R121 at (140.5, 87.4)
- removed the R121 at (169.0, 43.4)
- removed the R121 at (169.0, 87.4)
- removed the R121 at (140.5, 43.4)
- removed the R122 at (136.0, 34.2)
- removed the R122 at (164.5, 78.2)
- removed the R122 at (136.0, 78.2)
- removed the R122 at (164.5, 34.2)
- removed the R123 at (136.0, 76.2)
- removed the R123 at (164.5, 76.2)
- removed the R123 at (136.0, 32.2)
- removed the R123 at (164.5, 32.2)
- removed the R124 at (164.5, 80.4)
- removed the R124 at (164.5, 36.4)
- removed the R124 at (136.0, 80.4)
- removed the R124 at (136.0, 36.4)
- removed the R125 at (164.2, 102.7)
- removed the R125 at (135.7, 102.7)
- removed the R125 at (135.7, 58.7)
- removed the R125 at (164.2, 58.7)
- removed the R126 at (168.5, 75.6)
- removed the R126 at (168.5, 31.6)
- removed the R126 at (140.0, 31.6)
- removed the R126 at (140.0, 75.6)
- removed the R128 at (171.2, 41.2)
- removed the R128 at (142.7, 41.2)
- removed the R128 at (171.2, 85.2)
- removed the R128 at (142.7, 85.2)
- removed REF** (x4): Error, Error
- removed the SCL108 at (124.3, 105.0)
- removed the SCL108 at (152.8, 61.0)
- removed the SCL108 at (124.3, 61.0)
- removed the SCL108 at (152.8, 105.0)
- removed the SCL109 at (170.6, 87.0)
- removed the SCL109 at (170.6, 43.0)
- removed the SCL109 at (142.1, 87.0)
- removed the SCL109 at (142.1, 43.0)
- removed the SDA108 at (154.0, 62.2)
- removed the SDA108 at (125.5, 62.2)
- removed the SDA108 at (125.5, 106.2)
- removed the SDA108 at (154.0, 106.2)
- removed the T*C108 at (141.5, 75.7)
- removed the T*C108 at (170.0, 31.7)
- removed the T*C108 at (170.0, 75.7)
- removed the T*C108 at (141.5, 31.7)
- removed the T*C109 at (141.5, 77.6)
- removed the T*C109 at (170.0, 77.6)
- removed the T*C109 at (170.0, 33.6)
- removed the T*C109 at (141.5, 33.6)
- removed the T*C110 at (141.3, 83.4)
- removed the T*C110 at (141.3, 39.4)
- removed the T*C110 at (169.8, 39.4)
- removed the T*C110 at (169.8, 83.4)
- removed the TAC5212 at (134.5, 88.1)
- removed the TAC5212 at (162.9, 44.1)
- removed the TAC5212 at (134.5, 44.1)
- removed the TAC5212 at (162.9, 88.1)
- removed the U108 at (166.7, 101.8)
- removed the U108 at (166.7, 57.8)
- removed the U108 at (138.2, 57.8)
- removed the U108 at (138.2, 101.8)
- removed the U109 at (141.5, 36.6)
- removed the U109 at (141.5, 80.6)
- removed the U109 at (170.0, 36.6)
- removed the U109 at (170.0, 80.6)
- removed the board_outline108 at (147.5, 69.0)
- removed the board_outline108 at (176.0, 69.0)
- removed the board_outline108 at (147.5, 113.0)
- removed the board_outline108 at (176.0, 113.0)
- added 3V108: jumper, project_fp:jumper_slice_1mm, B.Cu at (139.2, 78.8)
- added 3V108: jumper, project_fp:jumper_slice_1mm, B.Cu at (166.7, 34.8)
- added 3V108: jumper, project_fp:jumper_slice_1mm, B.Cu at (139.2, 34.8)
- added 3V108: jumper, project_fp:jumper_slice_1mm, B.Cu at (166.7, 78.8)
- added 5V108: jumper, project_fp:jumper_slice_1mm, F.Cu at (172.4, 60.9)
- added 5V108: jumper, project_fp:jumper_slice_1mm, F.Cu at (172.4, 104.9)
- added 5V108: jumper, project_fp:jumper_slice_1mm, F.Cu at (144.9, 60.9)
- added 5V108: jumper, project_fp:jumper_slice_1mm, F.Cu at (144.9, 104.9)
- added ADD108: 0x50 | 0xA0, project_fp:SolderJumper-2_Open_Pad0.5x1.0mm_ADDR, F.Cu at (162.0, 36.8)
- added ADD108: 0x50 | 0xA0, project_fp:SolderJumper-2_Open_Pad0.5x1.0mm_ADDR, F.Cu at (162.0, 80.8)
- added ADD108: 0x50 | 0xA0, project_fp:SolderJumper-2_Open_Pad0.5x1.0mm_ADDR, F.Cu at (134.5, 36.8)
- added ADD108: 0x50 | 0xA0, project_fp:SolderJumper-2_Open_Pad0.5x1.0mm_ADDR, F.Cu at (134.5, 80.8)
- added ADD110: 0x52 | 0xA4, project_fp:SolderJumper-2_Open_Pad0.5x1.0mm_ADDR, F.Cu at (134.5, 77.6)
- added ADD110: 0x52 | 0xA4, project_fp:SolderJumper-2_Open_Pad0.5x1.0mm_ADDR, F.Cu at (162.0, 77.6)
- added ADD110: 0x52 | 0xA4, project_fp:SolderJumper-2_Open_Pad0.5x1.0mm_ADDR, F.Cu at (162.0, 33.6)
- added ADD110: 0x52 | 0xA4, project_fp:SolderJumper-2_Open_Pad0.5x1.0mm_ADDR, F.Cu at (134.5, 33.6)
- added ADD111: 0x53 | 0xA6, project_fp:SolderJumper-2_Open_Pad0.5x1.0mm_ADDR, F.Cu at (134.5, 76.0)
- added ADD111: 0x53 | 0xA6, project_fp:SolderJumper-2_Open_Pad0.5x1.0mm_ADDR, F.Cu at (162.0, 32.0)
- added ADD111: 0x53 | 0xA6, project_fp:SolderJumper-2_Open_Pad0.5x1.0mm_ADDR, F.Cu at (162.0, 76.0)
- added ADD111: 0x53 | 0xA6, project_fp:SolderJumper-2_Open_Pad0.5x1.0mm_ADDR, F.Cu at (134.5, 32.0)
- added ADD112: 0x51 | 0xA2, project_fp:SolderJumper-2_Open_Pad0.5x1.0mm_ADDR, F.Cu at (134.5, 35.2)
- added ADD112: 0x51 | 0xA2, project_fp:SolderJumper-2_Open_Pad0.5x1.0mm_ADDR, F.Cu at (162.0, 79.2)
- added ADD112: 0x51 | 0xA2, project_fp:SolderJumper-2_Open_Pad0.5x1.0mm_ADDR, F.Cu at (162.0, 35.2)
- added ADD112: 0x51 | 0xA2, project_fp:SolderJumper-2_Open_Pad0.5x1.0mm_ADDR, F.Cu at (134.5, 79.2)
- added C108: 10uF, project_fp:C_0805_2012Metric_Pad1.18x1.45mm_HandSolder, F.Cu at (133.5, 95.8)
- added C108: 10uF, project_fp:C_0805_2012Metric_Pad1.18x1.45mm_HandSolder, F.Cu at (133.5, 51.8)
- added C108: 10uF, project_fp:C_0805_2012Metric_Pad1.18x1.45mm_HandSolder, F.Cu at (161.0, 51.8)
- added C108: 10uF, project_fp:C_0805_2012Metric_Pad1.18x1.45mm_HandSolder, F.Cu at (161.0, 95.8)
- added C109: 0.1uF, project_fp:C_0402_1005Metric, F.Cu at (132.4, 92.6)
- added C109: 0.1uF, project_fp:C_0402_1005Metric, F.Cu at (159.9, 92.6)
- added C109: 0.1uF, project_fp:C_0402_1005Metric, F.Cu at (132.4, 48.6)
- added C109: 0.1uF, project_fp:C_0402_1005Metric, F.Cu at (159.9, 48.6)
- added C110: 47uF, project_fp:CP_EIA-3528-21_Kemet-B_Pad1.50x2.35mm_HandSolder, B.Cu at (166.0, 56.5)
- added C110: 47uF, project_fp:CP_EIA-3528-21_Kemet-B_Pad1.50x2.35mm_HandSolder, B.Cu at (166.0, 100.5)
- added C110: 47uF, project_fp:CP_EIA-3528-21_Kemet-B_Pad1.50x2.35mm_HandSolder, B.Cu at (138.5, 100.5)
- added C110: 47uF, project_fp:CP_EIA-3528-21_Kemet-B_Pad1.50x2.35mm_HandSolder, B.Cu at (138.5, 56.5)
- added C111: 10uF, project_fp:C_0805_2012Metric_Pad1.18x1.45mm_HandSolder, F.Cu at (169.3, 48.8)
- added C111: 10uF, project_fp:C_0805_2012Metric_Pad1.18x1.45mm_HandSolder, F.Cu at (169.3, 92.8)
- added C111: 10uF, project_fp:C_0805_2012Metric_Pad1.18x1.45mm_HandSolder, F.Cu at (141.8, 92.8)
- added C111: 10uF, project_fp:C_0805_2012Metric_Pad1.18x1.45mm_HandSolder, F.Cu at (141.8, 48.8)
- added C112: 0.1uF, project_fp:C_0402_1005Metric, F.Cu at (140.2, 45.6)
- added C112: 0.1uF, project_fp:C_0402_1005Metric, F.Cu at (140.2, 89.6)
- added C112: 0.1uF, project_fp:C_0402_1005Metric, F.Cu at (167.7, 89.6)
- added C112: 0.1uF, project_fp:C_0402_1005Metric, F.Cu at (167.7, 45.6)
- added C113: 0.047uF, project_fp:C_0603_1608Metric_Pad1.08x0.95mm_HandSolder, B.Cu at (131.6, 56.1)
- added C113: 0.047uF, project_fp:C_0603_1608Metric_Pad1.08x0.95mm_HandSolder, B.Cu at (131.6, 100.1)
- added C113: 0.047uF, project_fp:C_0603_1608Metric_Pad1.08x0.95mm_HandSolder, B.Cu at (159.1, 56.1)
- added C113: 0.047uF, project_fp:C_0603_1608Metric_Pad1.08x0.95mm_HandSolder, B.Cu at (159.1, 100.1)
- added C114: 47uF, project_fp:CP_EIA-3528-21_Kemet-B_Pad1.50x2.35mm_HandSolder, B.Cu at (138.5, 104.8)
- added C114: 47uF, project_fp:CP_EIA-3528-21_Kemet-B_Pad1.50x2.35mm_HandSolder, B.Cu at (138.5, 60.8)
- added C114: 47uF, project_fp:CP_EIA-3528-21_Kemet-B_Pad1.50x2.35mm_HandSolder, B.Cu at (166.0, 60.8)
- added C114: 47uF, project_fp:CP_EIA-3528-21_Kemet-B_Pad1.50x2.35mm_HandSolder, B.Cu at (166.0, 104.8)
- added C115: 10uF, project_fp:C_0805_2012Metric_Pad1.18x1.45mm_HandSolder, F.Cu at (137.3, 52.4)
- added C115: 10uF, project_fp:C_0805_2012Metric_Pad1.18x1.45mm_HandSolder, F.Cu at (137.3, 96.4)
- added C115: 10uF, project_fp:C_0805_2012Metric_Pad1.18x1.45mm_HandSolder, F.Cu at (164.8, 96.4)
- added C115: 10uF, project_fp:C_0805_2012Metric_Pad1.18x1.45mm_HandSolder, F.Cu at (164.8, 52.4)
- added C116: 0.1uF, project_fp:C_0402_1005Metric, F.Cu at (163.7, 49.4)
- added C116: 0.1uF, project_fp:C_0402_1005Metric, F.Cu at (136.2, 93.4)
- added C116: 0.1uF, project_fp:C_0402_1005Metric, F.Cu at (163.7, 93.4)
- added C116: 0.1uF, project_fp:C_0402_1005Metric, F.Cu at (136.2, 49.4)
- added C117: 0.047uF, project_fp:C_0603_1608Metric_Pad1.08x0.95mm_HandSolder, B.Cu at (159.1, 104.4)
- added C117: 0.047uF, project_fp:C_0603_1608Metric_Pad1.08x0.95mm_HandSolder, B.Cu at (131.6, 104.4)
- added C117: 0.047uF, project_fp:C_0603_1608Metric_Pad1.08x0.95mm_HandSolder, B.Cu at (159.1, 60.4)
- added C117: 0.047uF, project_fp:C_0603_1608Metric_Pad1.08x0.95mm_HandSolder, B.Cu at (131.6, 60.4)
- added C118: 1uF, project_fp:C_0603_1608Metric_Pad1.08x0.95mm_HandSolder, F.Cu at (127.8, 29.6)
- added C118: 1uF, project_fp:C_0603_1608Metric_Pad1.08x0.95mm_HandSolder, F.Cu at (127.8, 73.6)
- added C118: 1uF, project_fp:C_0603_1608Metric_Pad1.08x0.95mm_HandSolder, F.Cu at (155.3, 73.6)
- added C118: 1uF, project_fp:C_0603_1608Metric_Pad1.08x0.95mm_HandSolder, F.Cu at (155.3, 29.6)
- added C119: 1uF, project_fp:C_0603_1608Metric_Pad1.08x0.95mm_HandSolder, F.Cu at (162.5, 94.6)
- added C119: 1uF, project_fp:C_0603_1608Metric_Pad1.08x0.95mm_HandSolder, F.Cu at (135.0, 50.6)
- added C119: 1uF, project_fp:C_0603_1608Metric_Pad1.08x0.95mm_HandSolder, F.Cu at (135.0, 94.6)
- added C119: 1uF, project_fp:C_0603_1608Metric_Pad1.08x0.95mm_HandSolder, F.Cu at (162.5, 50.6)
- added C120: 47uF, project_fp:CP_EIA-3528-21_Kemet-B_Pad1.50x2.35mm_HandSolder, B.Cu at (138.5, 52.2)
- added C120: 47uF, project_fp:CP_EIA-3528-21_Kemet-B_Pad1.50x2.35mm_HandSolder, B.Cu at (138.5, 96.2)
- added C120: 47uF, project_fp:CP_EIA-3528-21_Kemet-B_Pad1.50x2.35mm_HandSolder, B.Cu at (166.0, 96.2)
- added C120: 47uF, project_fp:CP_EIA-3528-21_Kemet-B_Pad1.50x2.35mm_HandSolder, B.Cu at (166.0, 52.2)
- added C121: 0.047uF, project_fp:C_0603_1608Metric_Pad1.08x0.95mm_HandSolder, B.Cu at (131.6, 51.8)
- added C121: 0.047uF, project_fp:C_0603_1608Metric_Pad1.08x0.95mm_HandSolder, B.Cu at (131.6, 95.8)
- added C121: 0.047uF, project_fp:C_0603_1608Metric_Pad1.08x0.95mm_HandSolder, B.Cu at (159.1, 51.8)
- added C121: 0.047uF, project_fp:C_0603_1608Metric_Pad1.08x0.95mm_HandSolder, B.Cu at (159.1, 95.8)
- added C122: 47uF, project_fp:CP_EIA-3528-21_Kemet-B_Pad1.50x2.35mm_HandSolder, B.Cu at (166.9, 47.1)
- added C122: 47uF, project_fp:CP_EIA-3528-21_Kemet-B_Pad1.50x2.35mm_HandSolder, B.Cu at (166.9, 91.1)
- added C122: 47uF, project_fp:CP_EIA-3528-21_Kemet-B_Pad1.50x2.35mm_HandSolder, B.Cu at (139.4, 47.1)
- added C122: 47uF, project_fp:CP_EIA-3528-21_Kemet-B_Pad1.50x2.35mm_HandSolder, B.Cu at (139.4, 91.1)
- added C123: 0.047uF, project_fp:C_0603_1608Metric_Pad1.08x0.95mm_HandSolder, B.Cu at (159.1, 47.9)
- added C123: 0.047uF, project_fp:C_0603_1608Metric_Pad1.08x0.95mm_HandSolder, B.Cu at (131.6, 47.9)
- added C123: 0.047uF, project_fp:C_0603_1608Metric_Pad1.08x0.95mm_HandSolder, B.Cu at (159.1, 91.9)
- added C123: 0.047uF, project_fp:C_0603_1608Metric_Pad1.08x0.95mm_HandSolder, B.Cu at (131.6, 91.9)
- added C124: 10UF, project_fp:C_0603_1608Metric_Pad1.08x0.95mm_HandSolder, B.Cu at (135.0, 31.0)
- added C124: 10UF, project_fp:C_0603_1608Metric_Pad1.08x0.95mm_HandSolder, B.Cu at (162.5, 75.0)
- added C124: 10UF, project_fp:C_0603_1608Metric_Pad1.08x0.95mm_HandSolder, B.Cu at (162.5, 31.0)
- added C124: 10UF, project_fp:C_0603_1608Metric_Pad1.08x0.95mm_HandSolder, B.Cu at (135.0, 75.0)
- added C125: 10UF, project_fp:C_0603_1608Metric_Pad1.08x0.95mm_HandSolder, B.Cu at (162.6, 33.6)
- added C125: 10UF, project_fp:C_0603_1608Metric_Pad1.08x0.95mm_HandSolder, B.Cu at (135.1, 33.6)
- added C125: 10UF, project_fp:C_0603_1608Metric_Pad1.08x0.95mm_HandSolder, B.Cu at (135.1, 77.6)
- added C125: 10UF, project_fp:C_0603_1608Metric_Pad1.08x0.95mm_HandSolder, B.Cu at (162.6, 77.6)
- added C126: 10UF, project_fp:C_0603_1608Metric_Pad1.08x0.95mm_HandSolder, B.Cu at (162.5, 37.2)
- added C126: 10UF, project_fp:C_0603_1608Metric_Pad1.08x0.95mm_HandSolder, B.Cu at (135.0, 37.2)
- added C126: 10UF, project_fp:C_0603_1608Metric_Pad1.08x0.95mm_HandSolder, B.Cu at (135.0, 81.2)
- added C126: 10UF, project_fp:C_0603_1608Metric_Pad1.08x0.95mm_HandSolder, B.Cu at (162.5, 81.2)
- added C127: 10UF, project_fp:C_0603_1608Metric_Pad1.08x0.95mm_HandSolder, B.Cu at (135.0, 83.9)
- added C127: 10UF, project_fp:C_0603_1608Metric_Pad1.08x0.95mm_HandSolder, B.Cu at (162.5, 83.9)
- added C127: 10UF, project_fp:C_0603_1608Metric_Pad1.08x0.95mm_HandSolder, B.Cu at (135.0, 39.9)
- added C127: 10UF, project_fp:C_0603_1608Metric_Pad1.08x0.95mm_HandSolder, B.Cu at (162.5, 39.9)
- added C128: 1uF, project_fp:C_0603_1608Metric_Pad1.08x0.95mm_HandSolder, F.Cu at (141.6, 101.0)
- added C128: 1uF, project_fp:C_0603_1608Metric_Pad1.08x0.95mm_HandSolder, F.Cu at (169.1, 57.0)
- added C128: 1uF, project_fp:C_0603_1608Metric_Pad1.08x0.95mm_HandSolder, F.Cu at (169.1, 101.0)
- added C128: 1uF, project_fp:C_0603_1608Metric_Pad1.08x0.95mm_HandSolder, F.Cu at (141.6, 57.0)
- added C129: 1uF, project_fp:C_0603_1608Metric_Pad1.08x0.95mm_HandSolder, B.Cu at (167.8, 85.5)
- added C129: 1uF, project_fp:C_0603_1608Metric_Pad1.08x0.95mm_HandSolder, B.Cu at (167.8, 41.5)
- added C129: 1uF, project_fp:C_0603_1608Metric_Pad1.08x0.95mm_HandSolder, B.Cu at (140.4, 85.5)
- added C129: 1uF, project_fp:C_0603_1608Metric_Pad1.08x0.95mm_HandSolder, B.Cu at (140.4, 41.5)
- added C130: 47uF, project_fp:C_0805_2012Metric_Pad1.15x1.40mm_HandSolder, B.Cu at (143.0, 104.6)
- added C130: 47uF, project_fp:C_0805_2012Metric_Pad1.15x1.40mm_HandSolder, B.Cu at (170.5, 60.6)
- added C130: 47uF, project_fp:C_0805_2012Metric_Pad1.15x1.40mm_HandSolder, B.Cu at (143.0, 60.6)
- added C130: 47uF, project_fp:C_0805_2012Metric_Pad1.15x1.40mm_HandSolder, B.Cu at (170.5, 104.6)
- added C131: 47uF, project_fp:C_0805_2012Metric_Pad1.15x1.40mm_HandSolder, B.Cu at (172.7, 60.6)
- added C131: 47uF, project_fp:C_0805_2012Metric_Pad1.15x1.40mm_HandSolder, B.Cu at (145.2, 104.6)
- added C131: 47uF, project_fp:C_0805_2012Metric_Pad1.15x1.40mm_HandSolder, B.Cu at (145.2, 60.6)
- added C131: 47uF, project_fp:C_0805_2012Metric_Pad1.15x1.40mm_HandSolder, B.Cu at (172.7, 104.6)
- added D108: TPD1E1B04 - 0402 size, project_fp:D_0402_1005Metric_Pad0.77x0.64mm_HandSolder, B.Cu at (156.2, 100.9)
- added D108: TPD1E1B04 - 0402 size, project_fp:D_0402_1005Metric_Pad0.77x0.64mm_HandSolder, B.Cu at (156.2, 56.9)
- added D108: TPD1E1B04 - 0402 size, project_fp:D_0402_1005Metric_Pad0.77x0.64mm_HandSolder, B.Cu at (128.7, 56.9)
- added D108: TPD1E1B04 - 0402 size, project_fp:D_0402_1005Metric_Pad0.77x0.64mm_HandSolder, B.Cu at (128.7, 100.9)
- added D109: TPD1E1B04 - 0402 size, project_fp:D_0402_1005Metric_Pad0.77x0.64mm_HandSolder, B.Cu at (128.7, 105.2)
- added D109: TPD1E1B04 - 0402 size, project_fp:D_0402_1005Metric_Pad0.77x0.64mm_HandSolder, B.Cu at (128.7, 61.2)
- added D109: TPD1E1B04 - 0402 size, project_fp:D_0402_1005Metric_Pad0.77x0.64mm_HandSolder, B.Cu at (156.2, 61.2)
- added D109: TPD1E1B04 - 0402 size, project_fp:D_0402_1005Metric_Pad0.77x0.64mm_HandSolder, B.Cu at (156.2, 105.2)
- added D110: TPD1E1B04 - 0402 size, project_fp:D_0402_1005Metric_Pad0.77x0.64mm_HandSolder, B.Cu at (156.2, 96.6)
- added D110: TPD1E1B04 - 0402 size, project_fp:D_0402_1005Metric_Pad0.77x0.64mm_HandSolder, B.Cu at (128.7, 96.6)
- added D110: TPD1E1B04 - 0402 size, project_fp:D_0402_1005Metric_Pad0.77x0.64mm_HandSolder, B.Cu at (156.2, 52.6)
- added D110: TPD1E1B04 - 0402 size, project_fp:D_0402_1005Metric_Pad0.77x0.64mm_HandSolder, B.Cu at (128.7, 52.6)
- added D111: TPD1E1B04 - 0402 size, project_fp:D_0402_1005Metric_Pad0.77x0.64mm_HandSolder, B.Cu at (156.2, 48.9)
- added D111: TPD1E1B04 - 0402 size, project_fp:D_0402_1005Metric_Pad0.77x0.64mm_HandSolder, B.Cu at (128.7, 48.9)
- added D111: TPD1E1B04 - 0402 size, project_fp:D_0402_1005Metric_Pad0.77x0.64mm_HandSolder, B.Cu at (128.7, 92.9)
- added D111: TPD1E1B04 - 0402 size, project_fp:D_0402_1005Metric_Pad0.77x0.64mm_HandSolder, B.Cu at (156.2, 92.9)
- added D112: TPD1E1B04 - 0402 size, project_fp:D_0402_1005Metric_Pad0.77x0.64mm_HandSolder, B.Cu at (128.7, 30.2)
- added D112: TPD1E1B04 - 0402 size, project_fp:D_0402_1005Metric_Pad0.77x0.64mm_HandSolder, B.Cu at (128.7, 74.2)
- added D112: TPD1E1B04 - 0402 size, project_fp:D_0402_1005Metric_Pad0.77x0.64mm_HandSolder, B.Cu at (156.1, 30.2)
- added D112: TPD1E1B04 - 0402 size, project_fp:D_0402_1005Metric_Pad0.77x0.64mm_HandSolder, B.Cu at (156.1, 74.2)
- added D113: TPD1E1B04 - 0402 size, project_fp:D_0402_1005Metric_Pad0.77x0.64mm_HandSolder, B.Cu at (128.6, 33.8)
- added D113: TPD1E1B04 - 0402 size, project_fp:D_0402_1005Metric_Pad0.77x0.64mm_HandSolder, B.Cu at (128.6, 77.8)
- added D113: TPD1E1B04 - 0402 size, project_fp:D_0402_1005Metric_Pad0.77x0.64mm_HandSolder, B.Cu at (156.1, 77.8)
- added D113: TPD1E1B04 - 0402 size, project_fp:D_0402_1005Metric_Pad0.77x0.64mm_HandSolder, B.Cu at (156.1, 33.8)
- added D114: TPD1E1B04 - 0402 size, project_fp:D_0402_1005Metric_Pad0.77x0.64mm_HandSolder, B.Cu at (156.1, 81.4)
- added D114: TPD1E1B04 - 0402 size, project_fp:D_0402_1005Metric_Pad0.77x0.64mm_HandSolder, B.Cu at (156.1, 37.4)
- added D114: TPD1E1B04 - 0402 size, project_fp:D_0402_1005Metric_Pad0.77x0.64mm_HandSolder, B.Cu at (128.6, 81.4)
- added D114: TPD1E1B04 - 0402 size, project_fp:D_0402_1005Metric_Pad0.77x0.64mm_HandSolder, B.Cu at (128.6, 37.4)
- added D115: TPD1E1B04 - 0402 size, project_fp:D_0402_1005Metric_Pad0.77x0.64mm_HandSolder, B.Cu at (156.0, 85.0)
- added D115: TPD1E1B04 - 0402 size, project_fp:D_0402_1005Metric_Pad0.77x0.64mm_HandSolder, B.Cu at (156.0, 41.0)
- added D115: TPD1E1B04 - 0402 size, project_fp:D_0402_1005Metric_Pad0.77x0.64mm_HandSolder, B.Cu at (128.5, 85.0)
- added D115: TPD1E1B04 - 0402 size, project_fp:D_0402_1005Metric_Pad0.77x0.64mm_HandSolder, B.Cu at (128.5, 41.0)
- added D116: RED LED, project_fp:D_0805_2012Metric_custom, F.Cu at (168.2, 33.6)
- added D116: RED LED, project_fp:D_0805_2012Metric_custom, F.Cu at (140.7, 77.6)
- added D116: RED LED, project_fp:D_0805_2012Metric_custom, F.Cu at (168.2, 77.6)
- added D116: RED LED, project_fp:D_0805_2012Metric_custom, F.Cu at (140.7, 33.6)
- added DOUT108: Jump DOUT1, project_fp:jumper_slice_disconnected_alt-text, F.Cu at (139.0, 98.5)
- added DOUT108: Jump DOUT1, project_fp:jumper_slice_disconnected_alt-text, F.Cu at (166.5, 98.5)
- added DOUT108: Jump DOUT1, project_fp:jumper_slice_disconnected_alt-text, F.Cu at (166.5, 54.5)
- added DOUT108: Jump DOUT1, project_fp:jumper_slice_disconnected_alt-text, F.Cu at (139.0, 54.5)
- added E108: jumper, project_fp:jumper_slice, F.Cu at (150.8, 98.1)
- added E108: jumper, project_fp:jumper_slice, F.Cu at (123.3, 54.1)
- added E108: jumper, project_fp:jumper_slice, F.Cu at (123.3, 98.1)
- added E108: jumper, project_fp:jumper_slice, F.Cu at (150.8, 54.1)
- added E109: jumper, project_fp:jumper_slice, F.Cu at (150.8, 31.7)
- added E109: jumper, project_fp:jumper_slice, F.Cu at (123.3, 75.7)
- added E109: jumper, project_fp:jumper_slice, F.Cu at (150.8, 75.7)
- added E109: jumper, project_fp:jumper_slice, F.Cu at (123.3, 31.7)
- added FB108: BLM21A601S - BLM21AG601SH1, project_fp:C_0805_2012Metric_Pad1.18x1.45mm_HandSolder, B.Cu at (158.8, 74.3)
- added FB108: BLM21A601S - BLM21AG601SH1, project_fp:C_0805_2012Metric_Pad1.18x1.45mm_HandSolder, B.Cu at (131.4, 30.3)
- added FB108: BLM21A601S - BLM21AG601SH1, project_fp:C_0805_2012Metric_Pad1.18x1.45mm_HandSolder, B.Cu at (131.4, 74.3)
- added FB108: BLM21A601S - BLM21AG601SH1, project_fp:C_0805_2012Metric_Pad1.18x1.45mm_HandSolder, B.Cu at (158.8, 30.3)
- added FB109: BLM21A601S - BLM21AG601SH1, project_fp:C_0805_2012Metric_Pad1.18x1.45mm_HandSolder, B.Cu at (131.3, 77.9)
- added FB109: BLM21A601S - BLM21AG601SH1, project_fp:C_0805_2012Metric_Pad1.18x1.45mm_HandSolder, B.Cu at (158.8, 33.9)
- added FB109: BLM21A601S - BLM21AG601SH1, project_fp:C_0805_2012Metric_Pad1.18x1.45mm_HandSolder, B.Cu at (131.3, 33.9)
- added FB109: BLM21A601S - BLM21AG601SH1, project_fp:C_0805_2012Metric_Pad1.18x1.45mm_HandSolder, B.Cu at (158.8, 77.9)
- added FB110: BLM21A601S - BLM21AG601SH1, project_fp:C_0805_2012Metric_Pad1.18x1.45mm_HandSolder, B.Cu at (158.7, 81.5)
- added FB110: BLM21A601S - BLM21AG601SH1, project_fp:C_0805_2012Metric_Pad1.18x1.45mm_HandSolder, B.Cu at (131.3, 37.5)
- added FB110: BLM21A601S - BLM21AG601SH1, project_fp:C_0805_2012Metric_Pad1.18x1.45mm_HandSolder, B.Cu at (158.7, 37.5)
- added FB110: BLM21A601S - BLM21AG601SH1, project_fp:C_0805_2012Metric_Pad1.18x1.45mm_HandSolder, B.Cu at (131.3, 81.5)
- added FB111: BLM21A601S - BLM21AG601SH1, project_fp:C_0805_2012Metric_Pad1.18x1.45mm_HandSolder, B.Cu at (131.1, 41.1)
- added FB111: BLM21A601S - BLM21AG601SH1, project_fp:C_0805_2012Metric_Pad1.18x1.45mm_HandSolder, B.Cu at (158.6, 85.1)
- added FB111: BLM21A601S - BLM21AG601SH1, project_fp:C_0805_2012Metric_Pad1.18x1.45mm_HandSolder, B.Cu at (158.6, 41.1)
- added FB111: BLM21A601S - BLM21AG601SH1, project_fp:C_0805_2012Metric_Pad1.18x1.45mm_HandSolder, B.Cu at (131.1, 85.1)
- added G108: VIA, project_fp:via, F.Cu at (165.6, 38.0)
- added G108: VIA, project_fp:via, F.Cu at (165.6, 82.0)
- added G108: VIA, project_fp:via, F.Cu at (138.1, 82.0)
- added G108: VIA, project_fp:via, F.Cu at (138.1, 38.0)
- added G109: VIA, project_fp:via, F.Cu at (140.8, 98.6)
- added G109: VIA, project_fp:via, F.Cu at (168.3, 54.6)
- added G109: VIA, project_fp:via, F.Cu at (168.3, 98.6)
- added G109: VIA, project_fp:via, F.Cu at (140.8, 54.6)
- added G110: VIA, project_fp:via, F.Cu at (165.1, 80.7)
- added G110: VIA, project_fp:via, F.Cu at (137.6, 80.7)
- added G110: VIA, project_fp:via, F.Cu at (137.6, 36.7)
- added G110: VIA, project_fp:via, F.Cu at (165.1, 36.7)
- added G111: VIA, project_fp:via, F.Cu at (169.3, 61.8)
- added G111: VIA, project_fp:via, F.Cu at (141.8, 61.8)
- added G111: VIA, project_fp:via, F.Cu at (141.8, 105.8)
- added G111: VIA, project_fp:via, F.Cu at (169.3, 105.8)
- added G112: VIA, project_fp:via, F.Cu at (137.6, 35.4)
- added G112: VIA, project_fp:via, F.Cu at (165.1, 35.4)
- added G112: VIA, project_fp:via, F.Cu at (137.6, 79.4)
- added G112: VIA, project_fp:via, F.Cu at (165.1, 79.4)
- added G113: VIA, project_fp:via, F.Cu at (169.5, 51.6)
- added G113: VIA, project_fp:via, F.Cu at (142.0, 51.6)
- added G113: VIA, project_fp:via, F.Cu at (142.0, 95.6)
- added G113: VIA, project_fp:via, F.Cu at (169.5, 95.6)
- added G114: VIA, project_fp:via, F.Cu at (139.2, 30.8)
- added G114: VIA, project_fp:via, F.Cu at (166.7, 30.8)
- added G114: VIA, project_fp:via, F.Cu at (166.7, 74.8)
- added G114: VIA, project_fp:via, F.Cu at (139.2, 74.8)
- added G115: VIA, project_fp:via, F.Cu at (170.9, 48.8)
- added G115: VIA, project_fp:via, F.Cu at (170.9, 92.8)
- added G115: VIA, project_fp:via, F.Cu at (143.4, 92.8)
- added G115: VIA, project_fp:via, F.Cu at (143.4, 48.8)
- added G116: VIA, project_fp:via, F.Cu at (161.3, 27.9)
- added G116: VIA, project_fp:via, F.Cu at (161.3, 71.9)
- added G116: VIA, project_fp:via, F.Cu at (133.8, 27.9)
- added G116: VIA, project_fp:via, F.Cu at (133.8, 71.9)
- added G117: jumper, project_fp:jumper_slice, F.Cu at (145.6, 54.3)
- added G117: jumper, project_fp:jumper_slice, F.Cu at (173.1, 98.3)
- added G117: jumper, project_fp:jumper_slice, F.Cu at (145.6, 98.3)
- added G117: jumper, project_fp:jumper_slice, F.Cu at (173.1, 54.3)
- added G118: jumper, project_fp:jumper_slice, F.Cu at (146.2, 31.6)
- added G118: jumper, project_fp:jumper_slice, F.Cu at (146.2, 75.6)
- added G118: jumper, project_fp:jumper_slice, F.Cu at (173.7, 31.6)
- added G118: jumper, project_fp:jumper_slice, F.Cu at (173.7, 75.6)
- added G119: jumper, project_fp:jumper_slice, B.Cu at (139.2, 32.2)
- added G119: jumper, project_fp:jumper_slice, B.Cu at (166.7, 76.2)
- added G119: jumper, project_fp:jumper_slice, B.Cu at (139.2, 76.2)
- added G119: jumper, project_fp:jumper_slice, B.Cu at (166.7, 32.2)
- added GND108: BRIDGE, project_fp:jumper_slice, B.Cu at (156.1, 44.6)
- added GND108: BRIDGE, project_fp:jumper_slice, B.Cu at (128.6, 44.6)
- added GND108: BRIDGE, project_fp:jumper_slice, B.Cu at (128.6, 88.6)
- added GND108: BRIDGE, project_fp:jumper_slice, B.Cu at (156.1, 88.6)
- added INM1: Jump Filter, project_fp:jumper_slice_via, B.Cu at (130.5, 36.0)
- added INM1: Jump Filter, project_fp:jumper_slice_via, B.Cu at (157.9, 80.0)
- added INM1: Jump Filter, project_fp:jumper_slice_via, B.Cu at (130.5, 80.0)
- added INM1: Jump Filter, project_fp:jumper_slice_via, B.Cu at (157.9, 36.0)
- added INM2: Jump Filter, project_fp:jumper_slice_via, B.Cu at (130.6, 28.8)
- added INM2: Jump Filter, project_fp:jumper_slice_via, B.Cu at (158.0, 72.8)
- added INM2: Jump Filter, project_fp:jumper_slice_via, B.Cu at (130.6, 72.8)
- added INM2: Jump Filter, project_fp:jumper_slice_via, B.Cu at (158.0, 28.8)
- added INP1: Jump Filter, project_fp:jumper_slice_via, B.Cu at (158.0, 83.6)
- added INP1: Jump Filter, project_fp:jumper_slice_via, B.Cu at (158.0, 39.6)
- added INP1: Jump Filter, project_fp:jumper_slice_via, B.Cu at (130.5, 39.6)
- added INP1: Jump Filter, project_fp:jumper_slice_via, B.Cu at (130.5, 83.6)
- added INP2: Jump Filter, project_fp:jumper_slice_via, B.Cu at (130.5, 76.4)
- added INP2: Jump Filter, project_fp:jumper_slice_via, B.Cu at (130.5, 32.4)
- added INP2: Jump Filter, project_fp:jumper_slice_via, B.Cu at (158.0, 76.4)
- added INP2: Jump Filter, project_fp:jumper_slice_via, B.Cu at (158.0, 32.4)
- added KiKit_FID_B_1: Fiducial, Fiducial, B.Cu at (98.3, 16.0)
- added KiKit_FID_B_2: Fiducial, Fiducial, B.Cu at (198.7, 16.0)
- added KiKit_FID_B_3: Fiducial, Fiducial, B.Cu at (98.3, 124.0)
- added KiKit_FID_T_1: Fiducial, Fiducial, F.Cu at (98.3, 16.0)
- added KiKit_FID_T_2: Fiducial, Fiducial, F.Cu at (198.7, 16.0)
- added KiKit_FID_T_3: Fiducial, Fiducial, F.Cu at (98.3, 124.0)
- added MCLK108: jumper, Jumper:SolderJumper-2_P1.3mm_Open_Pad1.0x1.5mm, B.Cu at (150.5, 61.0)
- added MCLK108: jumper, Jumper:SolderJumper-2_P1.3mm_Open_Pad1.0x1.5mm, B.Cu at (123.0, 105.0)
- added MCLK108: jumper, Jumper:SolderJumper-2_P1.3mm_Open_Pad1.0x1.5mm, B.Cu at (150.5, 105.0)
- added MCLK108: jumper, Jumper:SolderJumper-2_P1.3mm_Open_Pad1.0x1.5mm, B.Cu at (123.0, 61.0)
- added NT108: NetTie_2, project_fp:NetTie-2_SMD_Pad0.2mm, B.Cu at (142.4, 30.2)
- added NT108: NetTie_2, project_fp:NetTie-2_SMD_Pad0.2mm, B.Cu at (142.4, 74.2)
- added NT108: NetTie_2, project_fp:NetTie-2_SMD_Pad0.2mm, B.Cu at (169.9, 30.2)
- added NT108: NetTie_2, project_fp:NetTie-2_SMD_Pad0.2mm, B.Cu at (169.9, 74.2)
- added NT109: NetTie_2, project_fp:NetTie-2_SMD_Pad0.2mm, F.Cu at (160.7, 93.2)
- added NT109: NetTie_2, project_fp:NetTie-2_SMD_Pad0.2mm, F.Cu at (133.2, 49.2)
- added NT109: NetTie_2, project_fp:NetTie-2_SMD_Pad0.2mm, F.Cu at (133.2, 93.2)
- added NT109: NetTie_2, project_fp:NetTie-2_SMD_Pad0.2mm, F.Cu at (160.7, 49.2)
- added OM1: Jump Filter, project_fp:jumper_slice_via_alt_text, B.Cu at (130.6, 105.8)
- added OM1: Jump Filter, project_fp:jumper_slice_via_alt_text, B.Cu at (130.6, 61.8)
- added OM1: Jump Filter, project_fp:jumper_slice_via_alt_text, B.Cu at (158.1, 61.8)
- added OM1: Jump Filter, project_fp:jumper_slice_via_alt_text, B.Cu at (158.1, 105.8)
- added OM2: Jump Filter, project_fp:jumper_slice_via, B.Cu at (130.3, 93.6)
- added OM2: Jump Filter, project_fp:jumper_slice_via, B.Cu at (157.8, 93.6)
- added OM2: Jump Filter, project_fp:jumper_slice_via, B.Cu at (130.3, 49.6)
- added OM2: Jump Filter, project_fp:jumper_slice_via, B.Cu at (157.8, 49.6)
- added OP1: Jump Filter, project_fp:jumper_slice_via, B.Cu at (158.1, 57.8)
- added OP1: Jump Filter, project_fp:jumper_slice_via, B.Cu at (130.6, 101.8)
- added OP1: Jump Filter, project_fp:jumper_slice_via, B.Cu at (130.6, 57.8)
- added OP1: Jump Filter, project_fp:jumper_slice_via, B.Cu at (158.1, 101.8)
- added OP2: Jump Filter, project_fp:jumper_slice_via, B.Cu at (130.5, 97.5)
- added OP2: Jump Filter, project_fp:jumper_slice_via, B.Cu at (130.5, 53.5)
- added OP2: Jump Filter, project_fp:jumper_slice_via, B.Cu at (158.0, 53.5)
- added OP2: Jump Filter, project_fp:jumper_slice_via, B.Cu at (158.0, 97.5)
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Other:
- outline, holes or cut-outs redrawn
- board text added: "jlcpcb_4x4_T-DSP_TAC5212"
